File: Hardware/voicemail-box/voicemail-box.kicad_pcb (KiCad board)
At the start: 2 copper layers, 68.6 x 53.3 mm, 17 parts, among them J1 Power, J2 Digital/PWM, J3 Analog, J4 Digital/PWM, J5 Conn_02x06_Top_Bottom, U1 ESP32-WROOM-32

Commit message: + gitignore ~ added existing pinout of sandbox tests
Parts:
- added C3: 100n, Capacitor_SMD:C_0805_2012Metric_Pad1.18x1.45mm_HandSolder, F.Cu at (203.0, 62.5)
- added CN1: ~, Connector_PinSocket_2.54mm:PinSocket_2x15_P2.54mm_Vertical, B.Cu at (150.8, 97.5)
- added CN2: ~, Connector_PinSocket_2.54mm:PinSocket_2x17_P2.54mm_Vertical, B.Cu at (145.7, 51.7)
- added CN3: ~, Connector_PinSocket_2.54mm:PinSocket_2x10_P2.54mm_Vertical, B.Cu at (118.8, 51.7)
- added CN4: ~, Connector_PinSocket_2.54mm:PinSocket_2x08_P2.54mm_Vertical, B.Cu at (127.9, 97.5)
- added RN3: 10k, Resistor_SMD:R_Array_Convex_4x0603, F.Cu at (203.4, 68.5)
- moved RN2 46.2 mm to (213.2, 62.5)
- moved C1 46.2 mm to (217.6, 61.6)
- moved C2 46.2 mm to (217.6, 64.6)
- moved RN1 46.2 mm to (209.0, 62.5)
- moved U1 43.9 mm to (236.5, 59.6)
Connections:
- net /*10 renamed /D10
- net /*11 renamed /D11
- net /*3 renamed /D3
- net /*5 renamed /D5
- net /*6 renamed /D6
- net /*9 renamed /D9
- net /12 renamed /D12
- net /13 renamed /D13
- net /2 renamed /D2
- net /4 renamed /D4
- net /7 renamed /D7
- net /8 renamed /D8
- net /RX/0 renamed /RX/D0
- net /TX/1 renamed /TX/D1
- C1 pad 1: VCC_ESP -> +3V3
- C2 pad 1: VCC_ESP -> +3V3
- J1 pad 2: /IOREF -> +3V3
- J2 pad 1: /SCL/A5 -> /SCL
- J2 pad 2: /SDA/A4 -> /SDA
- J3 pad 5: /SDA/A4 -> /A4
- J3 pad 6: /SCL/A5 -> /A5
- J5 pad 12: VCC_ESP -> +3V3
- J5 pad 6: VCC_ESP -> +3V3
- R1 pad 1: VCC_ESP -> +3V3
- R2 pad 1: VCC_ESP -> +3V3
- U1 pad 2: VCC_ESP -> +3V3

Commit message: ~ HW Configuration
Parts:
- moved J5 47.0 mm to (258.2, 99.5), turned to -90 degrees
- moved U1 24.8 mm to (250.6, 80.0)
- moved RN3 24.0 mm to (221.5, 84.3)
- moved C1 24.0 mm to (235.7, 77.4)
- moved C2 24.0 mm to (235.7, 80.4)
- moved C3 24.0 mm to (221.1, 78.3)
- moved RN1 24.0 mm to (227.1, 78.3)
- moved RN2 24.0 mm to (231.2, 78.3)
