File: Hardware/voicemail-box/pinout.kicad_sch (KiCad schematic)
At the start: 4 parts

Commit message: ~ HW Configuration
Changed lines of the file:
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@@
 	)
 	(no_connect
-		(at 134.62 99.06)
+		(at 119.38 119.38)
 	)
 	(no_connect
@@
 	)
 	(no_connect
-		(at 134.62 116.84)
+		(at 119.38 137.16)
 	)
 	(no_connect
@@
 	)
 	(no_connect
-		(at 134.62 96.52)
+		(at 119.38 116.84)
 	)
 	(no_connect
@@
 	)
 	(no_connect
-		(at 134.62 102.87)
+		(at 119.38 123.19)
 	)
 	(no_connect
@@
 	)
 	(no_connect
-		(at 134.62 111.76)
+		(at 119.38 132.08)
 	)
 	(no_connect
@@
 	)
 	(no_connect
-		(at 134.62 105.41)
-	)
-	(no_connect
-		(at 134.62 109.22)
+		(at 119.38 125.73)
+	)
+	(no_connect
+		(at 119.38 129.54)
 	)
 	(no_connect
@@
 	)
 	(no_connect
-		(at 134.62 114.3)
+		(at 119.38 134.62)
 	)
 	(bus_entry
@@
 	(wire
 		(pts
-			(xy 140.97 96.52) (xy 134.62 96.52)
+			(xy 125.73 116.84) (xy 119.38 116.84)
 		)
 		(stroke
@@
 	(wire
 		(pts
-			(xy 140.97 114.3) (xy 134.62 114.3)
+			(xy 125.73 134.62) (xy 119.38 134.62)
 		)
 		(stroke
@@
 	(wire
 		(pts
-			(xy 140.97 111.76) (xy 134.62 111.76)
+			(xy 125.73 132.08) (xy 119.38 132.08)
 		)
 		(stroke
@@
 	(wire
 		(pts
+			(xy 118.11 83.82) (xy 140.97 83.82)
+		)
+		(stroke
+			(width 0)
+			(type default)
+		)
+	)
+	(wire
+		(pts
 			(xy 55.88 55.88) (xy 55.88 63.5)
 		)
@@
 	(wire
 		(pts
-			(xy 140.97 116.84) (xy 134.62 116.84)
+			(xy 125.73 137.16) (xy 119.38 137.16)
 		)
 		(stroke
@@
 	(wire
 		(pts
-			(xy 140.97 105.41) (xy 134.62 105.41)
+			(xy 125.73 125.73) (xy 119.38 125.73)
 		)
 		(stroke
@@
 	(wire
 		(pts
+			(xy 118.11 86.36) (xy 140.97 86.36)
+		)
+		(stroke
+			(width 0)
+			(type default)
+		)
+	)
+	(wire
+		(pts
 			(xy 232.41 124.46) (xy 234.95 124.46)
 		)
@@
 	(wire
 		(pts
-			(xy 140.97 102.87) (xy 134.62 102.87)
+			(xy 125.73 123.19) (xy 119.38 123.19)
 		)
 		(stroke
@@
 	(wire
 		(pts
-			(xy 140.97 109.22) (xy 134.62 109.22)
+			(xy 118.11 91.44) (xy 140.97 91.44)
+		)
+		(stroke
+			(width 0)
+			(type default)
+		)
+	)
+	(wire
+		(pts
+			(xy 125.73 129.54) (xy 119.38 129.54)
 		)
 		(stroke
@@
 	(wire
 		(pts
+			(xy 118.11 88.9) (xy 140.97 88.9)
+		)
+		(stroke
+			(width 0)
+			(type default)
+		)
+	)
+	(wire
+		(pts
 			(xy 232.41 83.82) (xy 273.05 83.82)
 		)
@@
 	(wire
 		(pts
-			(xy 140.97 99.06) (xy 134.62 99.06)
+			(xy 125.73 119.38) (xy 119.38 119.38)
 		)
 		(stroke
@@
 		(pts
 			(xy 209.55 101.6) (xy 209.55 119.38)
+		)
+		(stroke
+			(width 0)
+			(type default)
+		)
+	)
+	(wire
+		(pts
+			(xy 118.11 81.28) (xy 140.97 81.28)
 		)
 		(stroke
@@
 		)
 	)
+	(label "NFC_SCK"
+		(at 118.11 86.36 0)
+		(effects
+			(font
+				(size 1.27 1.27)
+			)
+			(justify left bottom)
+		)
+	)
 	(label "D6"
 		(at 273.05 99.06 180)
@@
 		)
 	)
+	(label "NFC_MOSI"
+		(at 118.11 81.28 0)
+		(effects
+			(font
+				(size 1.27 1.27)
+			)
+			(justify left bottom)
+		)
+	)
 	(label "NFC_LED6"
 		(at 273.05 96.52 180)
@@
 		)
 	)
+	(label "NFC_MISO"
+		(at 118.11 83.82 0)
+		(effects
+			(font
+				(size 1.27 1.27)
+			)
+			(justify left bottom)
+		)
+	)
 	(label "SD_DET"
 		(at 109.22 76.2 180)
@@
 	)
 	(label "NFC_NSS"
+		(at 118.11 88.9 0)
+		(effects
+			(font
+				(size 1.27 1.27)
+			)
+			(justify left bottom)
+		)
+	)
+	(label "NFC_NSS"
 		(at 273.05 78.74 180)
 		(effects
@@
 		)
 	)
+	(label "NFC_INT"
+		(at 118.11 91.44 0)
+		(effects
+			(font
+				(size 1.27 1.27)
+			)
+			(justify left bottom)
+		)
+	)
 	(label "SD_CLK"
 		(at 118.11 73.66 0)
@@
 		)
 	)
+	(hierarchical_label "NFC_MOSI"
+		(shape bidirectional)
+		(at 140.97 81.28 0)
+		(effects
+			(font
+				(size 1.27 1.27)
+			)
+			(justify left)
+		)
+	)
 	(hierarchical_label "NSS"
 		(shape bidirectional)
-		(at 140.97 109.22 0)
+		(at 125.73 129.54 0)
+		(effects
+			(font
+				(size 1.27 1.27)
+			)
+			(justify left)
+		)
+	)
+	(hierarchical_label "NFC_NSS"
+		(shape bidirectional)
+		(at 140.97 88.9 0)
 		(effects
 			(font
@@
 		)
 	)
+	(hierarchical_label "NFC_MISO"
+		(shape bidirectional)
+		(at 140.97 83.82 0)
+		(effects
+			(font
+				(size 1.27 1.27)
+			)
+			(justify left)
+		)
+	)
 	(hierarchical_label "SD_DET"
 		(shape bidirectional)
@@
 	(hierarchical_label "RX"
 		(shape bidirectional)
-		(at 140.97 96.52 0)
+		(at 125.73 116.84 0)
 		(effects
 			(font
@@
 	(hierarchical_label "TX"
 		(shape bidirectional)
-		(at 140.97 99.06 0)
+		(at 125.73 119.38 0)
 		(effects
 			(font
@@
 	(hierarchical_label "INT"
 		(shape bidirectional)
-		(at 140.97 102.87 0)
+		(at 125.73 123.19 0)
 		(effects
 			(font
@@
 	(hierarchical_label "SCK"
 		(shape bidirectional)
-		(at 140.97 116.84 0)
+		(at 125.73 137.16 0)
 		(effects
 			(font
@@
 	(hierarchical_label "MISO"
 		(shape bidirectional)
-		(at 140.97 114.3 0)
+		(at 125.73 134.62 0)
 		(effects
 			(font
@@
 	(hierarchical_label "MOSI"
 		(shape bidirectional)
-		(at 140.97 111.76 0)
+		(at 125.73 132.08 0)
 		(effects
 			(font
@@
 		)
 	)
+	(hierarchical_label "NFC_INT"
+		(shape bidirectional)
+		(at 140.97 91.44 0)
+		(effects
+			(font
+				(size 1.27 1.27)
+			)
+			(justify left)
+		)
+	)
+	(hierarchical_label "NFC_SCK"
+		(shape bidirectional)
+		(at 140.97 86.36 0)
+		(effects
+			(font
+				(size 1.27 1.27)
+			)
+			(justify left)
+		)
+	)
 	(hierarchical_label "SELECT"
 		(shape bidirectional)
-		(at 140.97 105.41 0)
-		(effects
-			(font
+		(at 125.73 125.73 0)
+		(effects
+			(font

Commit message: ~working on first pcb-Draft
Parts:
- added CN5: Conn_02x08_Odd_Even, Connector_PinSocket_2.54mm:PinSocket_2x08_P2.54mm_Vertical, symbol Connector_Generic:Conn_02x08_Odd_Even
Other:
- note added: "Arduino Standard Connector sadly does'nt offer enough pins with advanced features such as: I2S, microSD, more SPI and so on... So less standard pinouts have to be used. -> lots of jumpers to make it configurable."
- note added: "Expansion Connector of: STM32F469I-DISCO"
- note added: "Orange Marked = Arduino UNO Standard Pinout Yellow Marked = Nucleo144 Expansion to Arduino Standard"
- moved on the sheet: CN1, CN2, CN3, CN4

Commit message: -
Connections:
- net NFC_MISO is gone; now on net MISO: CN3.12 (D12)
- net NFC_MOSI is gone; now on net MOSI: CN3.14 (D11)
- net NFC_NSS is gone; now on net NSS: CN3.16 (D10)
- net NFC_SCK is gone; now on net SCK: CN3.10 (D13)
- net RX/D0 is gone; now on net RX: CN2.16 (D0)
- net TX/D1 is gone; now on net TX: CN2.14 (D1)
- net +3.3V: now also CN5.1 (Pin_1)
- net GND: now also CN5.2 (Pin_2)
- net I2S2_BCLK: now reaches CN5.10 (Pin_10)
- net SPI1_NSS: now reaches CN5.11 (Pin_11)
- net I2S2_WCLK: now reaches CN5.12 (Pin_12)
- net I2S2_SDA: now reaches CN5.14 (Pin_14)
- net nRST: now reaches CN5.4 (Pin_4)
- net SPI1_MISO: now reaches CN5.5 (Pin_5)
- net I2S2_MCLK: now reaches CN5.6 (Pin_6)
- net SPI1_SCK: now reaches CN5.7 (Pin_7)
- net SPI1_MOSI: now reaches CN5.9 (Pin_9)
- net NFC_LED1 renamed I2S2_SDA_ext
- net SCL renamed I2C_SCL
- net SDA renamed I2C_SDA
- no-connect marks 84 -> 67
Other:
- moved on the sheet: CN1, CN4

Commit message: schematic draft
Parts:
- renumbered CN5 to CN201, CN4 to CN202, CN1 to CN203, CN3 to CN204, CN2 to CN205
Connections:
- net SPI2_MOSI: now reaches CN204.13 (D22)
- net SPI2_SCK: now reaches CN204.15 (D23)
- net SPI2_NSS: now reaches CN204.17 (D24)
- net SPI2_MISO: now reaches CN204.19 (D25)
- no-connect marks 67 -> 69
Changed lines of the file:
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@@
-	)
-	(no_connect
-		(at 209.55 52.07)
 	)
 	(no_connect
@@
 	)
 	(no_connect
+		(at 45.72 146.05)
+	)
+	(no_connect
 		(at 86.36 66.04)
 	)
@@
 	)
 	(no_connect
+		(at 33.02 156.21)
+	)
+	(no_connect
 		(at 229.87 102.87)
 	)
 	(no_connect
-		(at 209.55 46.99)
+		(at 33.02 153.67)
 	)
 	(no_connect
@@
 	)
 	(no_connect
-		(at 209.55 44.45)
-	)
-	(no_connect
 		(at 209.55 72.39)
 	)
@@
 	)
 	(no_connect
+		(at 45.72 156.21)
+	)
+	(no_connect
+		(at 72.39 132.08)
+	)
+	(no_connect
 		(at 86.36 96.52)
 	)
@@
 	)
 	(no_connect
+		(at 33.02 140.97)
+	)
+	(no_connect
 		(at 209.55 29.21)
-	)
-	(no_connect
-		(at 209.55 49.53)
 	)
 	(no_connect
@@
 	(wire
 		(pts
+			(xy 204.47 44.45) (xy 209.55 44.45)
+		)
+		(stroke
+			(width 0)
+			(type default)
+		)
+	)
+	(wire
+		(pts
 			(xy 229.87 67.31) (xy 270.51 67.31)
 		)
@@
 	(wire
 		(pts
+			(xy 204.47 46.99) (xy 209.55 46.99)
+		)
+		(stroke
+			(width 0)
+			(type default)
+		)
+	)
+	(wire
+		(pts
 			(xy 29.21 148.59) (xy 33.02 148.59)
 		)
@@
 	(wire
 		(pts
+			(xy 204.47 52.07) (xy 209.55 52.07)
+		)
+		(stroke
+			(width 0)
+			(type default)
+		)
+	)
+	(wire
+		(pts
 			(xy 86.36 43.18) (xy 116.84 43.18)
 		)
@@
 			(width 0)
 			(type solid)
+		)
+	)
+	(wire
+		(pts
+			(xy 204.47 49.53) (xy 209.55 49.53)
+		)
+		(stroke
+			(width 0)
+			(type default)
 		)
 	)
@@
 		)
 	)
-	(label "TX{slash}D1"
-		(at 270.51 80.01 180)
-		(effects
-			(font
-				(size 1.27 1.27)
-			)
-			(justify right bottom)
-		)
-	)
 	(label "D4"
 		(at 270.51 72.39 180)
@@
 		)
 	)
-	(label "NFC_MOSI"
-		(at 270.51 44.45 180)
-		(effects
-			(font
-				(size 1.27 1.27)
-			)
-			(justify right bottom)
-		)
-	)
-	(label "NFC_MISO"
-		(at 270.51 41.91 180)
-		(effects
-			(font
-				(size 1.27 1.27)
-			)
-			(justify right bottom)
-		)
-	)
 	(label "SD_CMD"
 		(at 116.84 43.18 180)
@@
 		)
 	)
-	(label "NFC_SCK"
-		(at 270.51 39.37 180)
-		(effects
-			(font
-				(size 1.27 1.27)
-			)
-			(justify right bottom)
-		)
-	)
 	(label "SD_DAT0"
 		(at 125.73 27.94 0)
@@
 		)
 	)
-	(label "NFC_NSS"
-		(at 270.51 46.99 180)
-		(effects
-			(font
-				(size 1.27 1.27)
-			)
-			(justify right bottom)
-		)
-	)
 	(label "NFC_LED2"
 		(at 31.75 71.12 0)
@@
 	(label "nRST"
 		(at 72.39 132.08 180)
-		(effects
-			(font
-				(size 1.27 1.27)
-			)
-			(justify right bottom)
-		)
-	)
-	(label "RX{slash}D0"
-		(at 270.51 82.55 180)
 		(effects
 			(font
@@
 		)
 	)
+	(hierarchical_label "SPI2_MOSI"
+		(shape bidirectional)
+		(at 204.47 44.45 180)
+		(effects
+			(font
+				(size 1.27 1.27)
+			)
+			(justify right)
+		)
+	)
 	(hierarchical_label "SD_CLK"
 		(shape bidirectional)
@@
 		)
 	)
+	(hierarchical_label "SPI2_SCK"
+		(shape bidirectional)
+		(at 204.47 46.99 180)
+		(effects
+			(font
+				(size 1.27 1.27)
+			)
+			(justify right)
+		)
+	)
 	(hierarchical_label "I2C_SCL"
 		(shape bidirectional)
@@
 		)
 	)
+	(hierarchical_label "SPI2_MISO"
+		(shape bidirectional)
+		(at 204.47 52.07 180)
+		(effects
+			(font
+				(size 1.27 1.27)
+			)
+			(justify right)
+		)
+	)
 	(hierarchical_label "SPI1_SCK"
 		(shape bidirectional)
@@
 		)
 	)
-	(hierarchical_label "SELECT"
+	(hierarchical_label "SPI2_NSS"
 		(shape bidirectional)
-		(at 144.78 147.32 180)
+		(at 204.47 49.53 180)
 		(effects
 			(font
@@
 		(dnp no)
 		(fields_autoplaced yes)
-		(property "Reference" "CN4"
+		(property "Reference" "CN202"
 			(at 76.2 25.4 0)
 			(effects
@@
 			(project "voicemail-box"
 				(path "/e63e39d7-6ac0-4ffd-8aa3-1841a4541b55/8a941d25-10cd-4745-a77d-5d96df86b042"
-					(reference "CN4")
+					(reference "CN202")
 					(unit 1)
 				)
@@
 		(dnp no)
 		(fields_autoplaced yes)
-		(property "Reference" "#PWR013"
+		(property "Reference" "#PWR0208"
 			(at 88.9 110.49 0)
 			(effects
@@
 			(project "voicemail-box"
 				(path "/e63e39d7-6ac0-4ffd-8aa3-1841a4541b55/8a941d25-10cd-4745-a77d-5d96df86b042"
-					(reference "#PWR013")
+					(reference "#PWR0208")
 					(unit 1)
 				)
@@
 		(on_board yes)
 		(dnp no)
-		(property "Reference" "CN1"
+		(property "Reference" "CN203"
 			(at 76.2 60.96 0)
 			(effects
@@
 			(project "voicemail-box"
 				(path "/e63e39d7-6ac0-4ffd-8aa3-1841a4541b55/8a941d25-10cd-4745-a77d-5d96df86b042"
-					(reference "CN1")
+					(reference "CN203")
 					(unit 1)
 				)
@@
 		(dnp no)
 		(fields_autoplaced yes)
-		(property "Reference" "#PWR01"
+		(property "Reference" "#PWR0203"
 			(at 53.34 29.21 0)
 			(effects
@@
 			(project ""
 				(path "/e63e39d7-6ac0-4ffd-8aa3-1841a4541b55/8a941d25-10cd-4745-a77d-5d96df86b042"
-					(reference "#PWR01")
+					(reference "#PWR0203")
 					(unit 1)
 				)
@@
 		(dnp no)
 		(fields_autoplaced yes)
-		(property "Reference" "#PWR030"
+		(property "Reference" "#PWR0202"
 			(at 54.61 138.43 0)
 			(effects
@@
 			(project "voicemail-box"
 				(path "/e63e39d7-6ac0-4ffd-8aa3-1841a4541b55/8a941d25-10cd-4745-a77d-5d96df86b042"
-					(reference "#PWR030")
+					(reference "#PWR0202")
 					(unit 1)
 				)
@@
 		(dnp no)
 		(fields_autoplaced yes)
-		(property "Reference" "CN2"
+		(property "Reference" "CN205"
 			(at 219.71 59.69 0)
 			(effects
@@
 			(project "voicemail-box"
 				(path "/e63e39d7-6ac0-4ffd-8aa3-1841a4541b55/8a941d25-10cd-4745-a77d-5d96df86b042"
-					(reference "CN2")
+					(reference "CN205")
 					(unit 1)
 				)
@@
 		(dnp no)
 		(fields_autoplaced yes)
-		(property "Reference" "#PWR06"
+		(property "Reference" "#PWR0207"
 			(at 63.5 110.49 0)
 			(effects
@@
 			(project "voicemail-box"
 				(path "/e63e39d7-6ac0-4ffd-8aa3-1841a4541b55/8a941d25-10cd-4745-a77d-5d96df86b042"
-					(reference "#PWR06")
+					(reference "#PWR0207")
 					(unit 1)
 				)
@@
 		(dnp no)
 		(fields_autoplaced yes)
-		(property "Reference" "CN5"
+		(property "Reference" "CN201"
 			(at 39.37 132.08 0)
 			(effects
@@
 			(project ""
 				(path "/e63e39d7-6ac0-4ffd-8aa3-1841a4541b55/8a941d25-10cd-4745-a77d-5d96df86b042"
-					(reference "CN5")
+					(reference "CN201")
 					(unit 1)
 				)
@@
 		(dnp no)
 		(fields_autoplaced yes)
-		(property "Reference" "#PWR02"
+		(property "Reference" "#PWR0204"
 			(at 58.42 29.21 0)
 			(effects
@@
 			(project ""
 				(path "/e63e39d7-6ac0-4ffd-8aa3-1841a4541b55/8a941d25-10cd-4745-a77d-5d96df86b042"
-					(reference "#PWR02")
+					(reference "#PWR0204")
 					(unit 1)
 				)
@@
 		(dnp no)
 		(fields_autoplaced yes)
-		(property "Reference" "#PWR017"
+		(property "Reference" "#PWR0209"
 			(at 207.01 116.84 0)
 			(effects
@@
 			(project "voicemail-box"
 				(path "/e63e39d7-6ac0-4ffd-8aa3-1841a4541b55/8a941d25-10cd-4745-a77d-5d96df86b042"
-					(reference "#PWR017")
+					(reference "#PWR0209")
 					(unit 1)
 				)
@@
 		(dnp no)
 		(fields_autoplaced yes)
-		(property "Reference" "#PWR04"
+		(property "Reference" "#PWR0205"
 			(at 63.5 29.21 0)
 			(effects
@@
 			(project ""
 				(path "/e63e39d7-6ac0-4ffd-8aa3-1841a4541b55/8a941d25-10cd-4745-a77d-5d96df86b042"
-					(reference "#PWR04")
+					(reference "#PWR0205")
 					(unit 1)
 				)
@@
 		(dnp no)
 		(fields_autoplaced yes)
-		(property "Reference" "#PWR031"
+		(property "Reference" "#PWR0201"
 			(at 34.29 138.43 0)
 			(effects
@@
 			(project "voicemail-box"
 				(path "/e63e39d7-6ac0-4ffd-8aa3-1841a4541b55/8a941d25-10cd-4745-a77d-5d96df86b042"
-					(reference "#PWR031")
+					(reference "#PWR0201")
 					(unit 1)
 				)
@@
 		(dnp no)
 		(fields_autoplaced yes)
-		(property "Reference" "#PWR018"
+		(property "Reference" "#PWR0211"
 			(at 232.41 116.84 0)
 			(effects
@@
 			(project "voicemail-box"
 				(path "/e63e39d7-6ac0-4ffd-8aa3-1841a4541b55/8a941d25-10cd-4745-a77d-5d96df86b042"
-					(reference "#PWR018")
+					(reference "#PWR0211")
 					(unit 1)
 				)
@@
 		(on_board yes)
 		(dnp no)
-		(property "Reference" "CN3"
+		(property "Reference" "CN204"
 			(at 219.71 21.59 0)
 			(effects
@@
 			(project "voicemail-box"
 				(path "/e63e39d7-6ac0-4ffd-8aa3-1841a4541b55/8a941d25-10cd-4745-a77d-5d96df86b042"
-					(reference "CN3")
+					(reference "CN204")
 					(unit 1)
 				)
@@
 		(dnp no)
 		(fields_autoplaced yes)
-		(property "Reference" "#PWR03"
+		(property "Reference" "#PWR0206"
 			(at 63.5 59.69 0)
 			(effects
@@
 			(project ""
 				(path "/e63e39d7-6ac0-4ffd-8aa3-1841a4541b55/8a941d25-10cd-4745-a77d-5d96df86b042"
-					(reference "#PWR03")
+					(reference "#PWR0206")
 					(unit 1)
 				)
@@
 		(dnp no)
 		(fields_autoplaced yes)
-		(property "Reference" "#PWR05"
+		(property "Reference" "#PWR0210"
 			(at 232.41 59.69 0)
 			(effects
@@
 			(project "voicemail-box"
 				(path "/e63e39d7-6ac0-4ffd-8aa3-1841a4541b55/8a941d25-10cd-4745-a77d-5d96df86b042"
-					(reference "#PWR05")
+					(reference "#PWR0210")
 					(unit 1)
 				)
