File: Hardware/voicemail-box/pinout.kicad_sch (KiCad schematic)
At the start: 5 parts, among them CN201 Conn_02x08_Odd_Even

Commit message: ~layout
Connections:
- net +3.3V renamed +3V3
- net VCC: no longer names the net of CN202.15 (VCC)

Commit message: state of pcb ordered
Connections:
- net BTN0: now also CN204.18 (D9)
- net BTN1: now also CN205.6 (D5)
- net BTN2: now also CN205.8 (D4)
- net BTN3: now also CN205.10 (D3)
- net CODEC_nRESET: now also CN205.12 (D2)
- net INT: now also CN203.9 (A4)
- net LED0: now also CN205.4 (D6)
- net LED1: now also CN205.2 (D7)
- net POT0: now also CN203.7 (A3)
- net POT1: now also CN203.5 (A2)
- no-connect marks 74 -> 54
