File: Hardware/voicemail-box/NFC_breakaway.kicad_sch (KiCad schematic)
At the start: 1 part, among them U2 ST25R3911B-AQF

Commit message: ~ HW Configuration
Parts:
- removed U2: ST25R3911B-AQF, Package_DFN_QFN:QFN-32-1EP_5x5mm_P0.5mm_EP3.6x3.6mm_ThermalVias, symbol RF_NFC:ST25R3911B-AQF
- added C10, C12, C16, C18, C20, C22, C6: 2u2, Capacitor_SMD:C_0201_0603Metric_Pad0.64x0.40mm_HandSolder, symbol Device:C
- added C11, C13, C15, C19, C21, C7, C8, C9: 10n, Capacitor_SMD:C_0201_0603Metric_Pad0.64x0.40mm_HandSolder, symbol Device:C
- added C14: 1u, Capacitor_SMD:C_0201_0603Metric_Pad0.64x0.40mm_HandSolder, symbol Device:C
- added C17: 22n, Capacitor_SMD:C_0201_0603Metric_Pad0.64x0.40mm_HandSolder, symbol Device:C
- added C23, C24: 10p, Capacitor_SMD:C_0201_0603Metric_Pad0.64x0.40mm_HandSolder, symbol Device:C
- added R4: np_0R, Resistor_SMD:R_0805_2012Metric_Pad1.20x1.40mm_HandSolder, symbol Device:R
- added R5: 0R, Resistor_SMD:R_0805_2012Metric_Pad1.20x1.40mm_HandSolder, symbol Device:R
- added U2: ST25R3916B, symbol myParts:ST25R3916B
- added Y1: 27.12Mhz, symbol Device:Crystal_GND24
Connections:
- new net: R4.2, R5.1, U2.20 (I2C_EN)
- new net: C24.1, U2.4 (XTO), Y1.3
- new net: C23.1, U2.5 (XTI), Y1.1
- new net: C15.1, C16.1, C19.1, C20.1, U2.14 (VDD_DR), U2.9 (VDD_RF)
- new net: C10.1, C9.1, U2.7 (VDD_A)
- new net: C13.1, C14.1, U2.24 (AGDC)
- new net: C17.1, C18.1, U2.11 (VDD_AM)
- new net +3V3: C8.1, U2.1 (VDD_IO)
- new net GND: C10.2, C11.2, C12.2, C13.2, C14.2, C15.2, C16.2, C17.2, C18.2, C19.2, C20.2, C21.2, C22.2, C23.2, C24.2, C6.2, C7.2, C8.2, C9.2, R5.2, U2.12 (GND_DR), U2.16 (GND_DR), U2.21 (VSS), U2.26 (GND_A), U2.33 (EP), U2.6 (GND_D), Y1.2, Y1.4
- new net VDD_D: C6.1, C7.1, R4.1, U2.3 (VDD_D)
- new net V_RF: C11.1, C12.1, C21.1, C22.1, U2.10 (VDD_TX), U2.8 (VDD)
- no-connect marks 0 -> 3

Commit message: ~working on first pcb-Draft
Parts:
- U2: footprint (none) -> Package_DFN_QFN:UFQFPN-32-1EP_5x5mm_P0.5mm_EP3.5x3.5mm
- Y1: footprint (none) -> Crystal:Crystal_SMD_SeikoEpson_FA128-4Pin_2.0x1.6mm
Connections:
- net NFC_INT: now also U2.27 (IRQ)
- net NFC_MISO: now also U2.32 (MISO)
- net NFC_MOSI: now also U2.31 (MOSI)
- net NFC_NSS: now also U2.29 (/SS)
- net NFC_SCK: now also U2.30 (SCLK)
Changed lines of the file:
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@@
 	(wire
 		(pts
-			(xy 60.96 66.04) (xy 38.1 66.04)
+			(xy 72.39 52.07) (xy 95.25 52.07)
 		)
 		(stroke
@@
 	(wire
 		(pts
-			(xy 60.96 60.96) (xy 38.1 60.96)
+			(xy 72.39 62.23) (xy 95.25 62.23)
 		)
 		(stroke
@@
 	(wire
 		(pts
-			(xy 60.96 58.42) (xy 38.1 58.42)
+			(xy 72.39 67.31) (xy 95.25 67.31)
 		)
 		(stroke
@@
 	(wire
 		(pts
-			(xy 60.96 55.88) (xy 38.1 55.88)
+			(xy 72.39 64.77) (xy 95.25 64.77)
 		)
 		(stroke
@@
 	(wire
 		(pts
-			(xy 60.96 63.5) (xy 38.1 63.5)
+			(xy 72.39 59.69) (xy 95.25 59.69)
 		)
 		(stroke
@@
 	)
 	(label "NFC_INT"
-		(at 60.96 66.04 180)
+		(at 86.36 52.07 180)
 		(effects
 			(font
@@
 	)
 	(label "NFC_MOSI"
-		(at 60.96 55.88 180)
+		(at 86.36 64.77 180)
 		(effects
 			(font
@@
 	)
 	(label "NFC_SCK"
-		(at 60.96 60.96 180)
+		(at 86.36 62.23 180)
 		(effects
 			(font
@@
 	)
 	(label "NFC_MISO"
-		(at 60.96 58.42 180)
+		(at 86.36 67.31 180)
 		(effects
 			(font
@@
 	)
 	(label "NFC_NSS"
-		(at 60.96 63.5 180)
+		(at 86.36 59.69 180)
 		(effects
 			(font
@@
 	(hierarchical_label "NFC_MISO"
 		(shape bidirectional)
-		(at 38.1 58.42 180)
+		(at 72.39 67.31 180)
 		(effects
 			(font
@@
 	(hierarchical_label "NFC_SCK"
 		(shape bidirectional)
-		(at 38.1 60.96 180)
+		(at 72.39 62.23 180)
 		(effects
 			(font
@@
 	(hierarchical_label "NFC_INT"
 		(shape bidirectional)
-		(at 38.1 66.04 180)
+		(at 72.39 52.07 180)
 		(effects
 			(font
@@
 	(hierarchical_label "NFC_MOSI"
 		(shape bidirectional)
-		(at 38.1 55.88 180)
+		(at 72.39 64.77 180)
 		(effects
 			(font
@@
 	(hierarchical_label "NFC_NSS"
 		(shape bidirectional)
-		(at 38.1 63.5 180)
+		(at 72.39 59.69 180)
 		(effects
 			(font
@@
 			)
 		)
-		(property "Footprint" ""
+		(property "Footprint" "Package_DFN_QFN:UFQFPN-32-1EP_5x5mm_P0.5mm_EP3.5x3.5mm"
 			(at 97.79 43.18 0)
 			(effects
@@
 			)
 		)
-		(property "Footprint" ""
+		(property "Footprint" "Package_DFN_QFN:UFQFPN-32-1EP_5x5mm_P0.5mm_EP3.5x3.5mm"
 			(at 33.02 119.38 0)
 			(effects
@@
 			)
 		)
-		(property "Footprint" ""
+		(property "Footprint" "Crystal:Crystal_SMD_SeikoEpson_FA128-4Pin_2.0x1.6mm"
 			(at 38.1 139.7 0)
 			(effects
@@
 			)
 		)
-		(property "Footprint" ""
+		(property "Footprint" "Package_DFN_QFN:UFQFPN-32-1EP_5x5mm_P0.5mm_EP3.5x3.5mm"
 			(at 153.67 43.18 0)
 			(effects
@@
 			)
 		)
-		(property "Footprint" ""
+		(property "Footprint" "Package_DFN_QFN:UFQFPN-32-1EP_5x5mm_P0.5mm_EP3.5x3.5mm"
 			(at 168.91 120.65 0)
 			(effects

Commit message: -
Parts:
- removed R5: 0R, Resistor_SMD:R_0805_2012Metric_Pad1.20x1.40mm_HandSolder, symbol Device:R
- added J8: Conn_01x02, Connector_PinHeader_2.54mm:PinHeader_1x02_P2.54mm_Vertical, symbol Connector_Generic:Conn_01x02
- R4: value np_0R -> 10k
Connections:
- net GND: now also J8.2 (Pin_2)
- net at R4.2, U2.20 (I2C_EN): now also J8.1 (Pin_1)
Other:
- moved on the sheet: R4, U2A, U2D

Commit message: schematic draft
Parts:
- removed J8: Conn_01x02, Connector_PinHeader_2.54mm:PinHeader_1x02_P2.54mm_Vertical, symbol Connector_Generic:Conn_01x02
- renumbered C24 to C501, C23 to C502, C8 to C503, C7 to C504, C6 to C505, C9 to C506, C10 to C507, C11 to C508, C12 to C509, C13 to C510, C14 to C511, C15 to C512, C16 to C513, C17 to C514, C18 to C515, C19 to C516, C20 to C517, C21 to C518, C22 to C519, R4 to R501, U2 to U501, Y1 to Y501
Connections:
- net I2C_Disable: now reaches R501.2, U501.20 (I2C_EN)
Other:
- note added: "Antenna Layout dependent"
- moved on the sheet: U501D

Commit message: HW Layout progress todo: + Antenna + Audio Jacks + Planes (Supply only)
Parts:
- C501, C502, C503, C504, C505, C506, C507, C508, C509, C510, C511, C512, C513, C514, C515, C516, C517, C518, C519: footprint Capacitor_SMD:C_0201_0603Metric_Pad0.64x0.40mm_HandSolder -> Capacitor_SMD:C_0603_1608Metric_Pad1.08x0.95mm_HandSolder
Changed lines of the file:
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@@
 			)
 		)
-		(property "Footprint" "Capacitor_SMD:C_0201_0603Metric_Pad0.64x0.40mm_HandSolder"
+		(property "Footprint" "Capacitor_SMD:C_0603_1608Metric_Pad1.08x0.95mm_HandSolder"
 			(at 27.6352 149.86 0)
 			(effects
@@
 			)
 		)
-		(property "Footprint" "Capacitor_SMD:C_0201_0603Metric_Pad0.64x0.40mm_HandSolder"
+		(property "Footprint" "Capacitor_SMD:C_0603_1608Metric_Pad1.08x0.95mm_HandSolder"
 			(at 50.4952 149.86 0)
 			(effects
@@
 			)
 		)
-		(property "Footprint" "Capacitor_SMD:C_0201_0603Metric_Pad0.64x0.40mm_HandSolder"
+		(property "Footprint" "Capacitor_SMD:C_0603_1608Metric_Pad1.08x0.95mm_HandSolder"
 			(at 209.2452 143.51 0)
 			(effects
@@
 			)
 		)
-		(property "Footprint" "Capacitor_SMD:C_0201_0603Metric_Pad0.64x0.40mm_HandSolder"
+		(property "Footprint" "Capacitor_SMD:C_0603_1608Metric_Pad1.08x0.95mm_HandSolder"
 			(at 113.9952 143.51 0)
 			(effects
@@
 			)
 		)
-		(property "Footprint" "Capacitor_SMD:C_0201_0603Metric_Pad0.64x0.40mm_HandSolder"
+		(property "Footprint" "Capacitor_SMD:C_0603_1608Metric_Pad1.08x0.95mm_HandSolder"
 			(at 93.6752 143.51 0)
 			(effects
@@
 			)
 		)
-		(property "Footprint" "Capacitor_SMD:C_0201_0603Metric_Pad0.64x0.40mm_HandSolder"
+		(property "Footprint" "Capacitor_SMD:C_0603_1608Metric_Pad1.08x0.95mm_HandSolder"
 			(at 260.0452 143.51 0)
 			(effects
@@
 			)
 		)
-		(property "Footprint" "Capacitor_SMD:C_0201_0603Metric_Pad0.64x0.40mm_HandSolder"
+		(property "Footprint" "Capacitor_SMD:C_0603_1608Metric_Pad1.08x0.95mm_HandSolder"
 			(at 154.6352 143.51 0)
 			(effects
@@
 			)
 		)
-		(property "Footprint" "Capacitor_SMD:C_0201_0603Metric_Pad0.64x0.40mm_HandSolder"
+		(property "Footprint" "Capacitor_SMD:C_0603_1608Metric_Pad1.08x0.95mm_HandSolder"
 			(at 73.3552 143.51 0)
 			(effects
@@
 			)
 		)
-		(property "Footprint" "Capacitor_SMD:C_0201_0603Metric_Pad0.64x0.40mm_HandSolder"
+		(property "Footprint" "Capacitor_SMD:C_0603_1608Metric_Pad1.08x0.95mm_HandSolder"
 			(at 134.3152 143.51 0)
 			(effects
@@
 			)
 		)
-		(property "Footprint" "Capacitor_SMD:C_0201_0603Metric_Pad0.64x0.40mm_HandSolder"
+		(property "Footprint" "Capacitor_SMD:C_0603_1608Metric_Pad1.08x0.95mm_HandSolder"
 			(at 239.7252 143.51 0)
 			(effects
@@
 			)
 		)
-		(property "Footprint" "Capacitor_SMD:C_0201_0603Metric_Pad0.64x0.40mm_HandSolder"
+		(property "Footprint" "Capacitor_SMD:C_0603_1608Metric_Pad1.08x0.95mm_HandSolder"
 			(at 83.5152 143.51 0)
 			(effects
@@
 			)
 		)
-		(property "Footprint" "Capacitor_SMD:C_0201_0603Metric_Pad0.64x0.40mm_HandSolder"
+		(property "Footprint" "Capacitor_SMD:C_0603_1608Metric_Pad1.08x0.95mm_HandSolder"
 			(at 219.4052 143.51 0)
 			(effects
@@
 			)
 		)
-		(property "Footprint" "Capacitor_SMD:C_0201_0603Metric_Pad0.64x0.40mm_HandSolder"
+		(property "Footprint" "Capacitor_SMD:C_0603_1608Metric_Pad1.08x0.95mm_HandSolder"
 			(at 229.5652 143.51 0)
 			(effects
@@
 			)
 		)
-		(property "Footprint" "Capacitor_SMD:C_0201_0603Metric_Pad0.64x0.40mm_HandSolder"
+		(property "Footprint" "Capacitor_SMD:C_0603_1608Metric_Pad1.08x0.95mm_HandSolder"
 			(at 249.8852 143.51 0)
 			(effects
@@
 			)
 		)
-		(property "Footprint" "Capacitor_SMD:C_0201_0603Metric_Pad0.64x0.40mm_HandSolder"
+		(property "Footprint" "Capacitor_SMD:C_0603_1608Metric_Pad1.08x0.95mm_HandSolder"
 			(at 144.4752 143.51 0)
 			(effects
@@
 			)
 		)
-		(property "Footprint" "Capacitor_SMD:C_0201_0603Metric_Pad0.64x0.40mm_HandSolder"
+		(property "Footprint" "Capacitor_SMD:C_0603_1608Metric_Pad1.08x0.95mm_HandSolder"
 			(at 103.8352 143.51 0)
 			(effects
@@
 			)
 		)
-		(property "Footprint" "Capacitor_SMD:C_0201_0603Metric_Pad0.64x0.40mm_HandSolder"
+		(property "Footprint" "Capacitor_SMD:C_0603_1608Metric_Pad1.08x0.95mm_HandSolder"
 			(at 199.0852 143.51 0)
 			(effects
@@
 			)
 		)
-		(property "Footprint" "Capacitor_SMD:C_0201_0603Metric_Pad0.64x0.40mm_HandSolder"
+		(property "Footprint" "Capacitor_SMD:C_0603_1608Metric_Pad1.08x0.95mm_HandSolder"
 			(at 270.2052 143.51 0)
 			(effects
@@
 			)
 		)
-		(property "Footprint" "Capacitor_SMD:C_0201_0603Metric_Pad0.64x0.40mm_HandSolder"
+		(property "Footprint" "Capacitor_SMD:C_0603_1608Metric_Pad1.08x0.95mm_HandSolder"
 			(at 124.1552 143.51 0)
 			(effects

Commit message: schema review
Parts:
- added C520, C521: 100p, Capacitor_SMD:C_0603_1608Metric_Pad1.08x0.95mm_HandSolder, symbol Device:C
- added C522, C523: 680p, Capacitor_SMD:C_0603_1608Metric_Pad1.08x0.95mm_HandSolder, symbol Device:C
- added C524, C525, C526: 47p, Capacitor_SMD:C_0603_1608Metric_Pad1.08x0.95mm_HandSolder, symbol Device:C
- added C527, C528: 56p, Capacitor_SMD:C_0603_1608Metric_Pad1.08x0.95mm_HandSolder, symbol Device:C
- added C531, C533: 10p, Capacitor_SMD:C_0603_1608Metric_Pad1.08x0.95mm_HandSolder, symbol Device:C
- added C532, C534: 180p, Capacitor_SMD:C_0603_1608Metric_Pad1.08x0.95mm_HandSolder, symbol Device:C
- added D502: BAV70W, Package_TO_SOT_SMD:SOT-23-3, symbol Device:D_Dual_CommonCathode_AAK_Parallel
- added J501: Conn_01x02, Connector_PinHeader_1.27mm:PinHeader_1x02_P1.27mm_Vertical, symbol Connector_Generic:Conn_01x02
- added L501, L502: 270n, symbol Device:L
- added Q501: NX3008NBK, Package_TO_SOT_SMD:SOT-23-3, symbol Simulation_SPICE:NMOS
- added R502: 47k, Resistor_SMD:R_0805_2012Metric_Pad1.20x1.40mm_HandSolder, symbol Device:R
- added R503, R504: 2k4, Resistor_SMD:R_0805_2012Metric_Pad1.20x1.40mm_HandSolder, symbol Device:R
- added R505: 100R, Resistor_SMD:R_0805_2012Metric_Pad1.20x1.40mm_HandSolder, symbol Device:R
- added U502, U503, U504, U505, U506: LXRW0YV600-054, LXRW0_MUR, symbol additial parts:LXRW0YV600-054
Connections:
- net GND: now also C522.1, C523.2, C527.2, C528.1, C532.1, C534.1, Q501.3 (S), R502.2, U502.2 (VT), U503.1 (GND), U504.1 (GND), U505.1 (GND), U506.1 (GND)
- net RFIO1: now reaches U501.13 (RFO1)
- net RFIO1: now also J501.1 (Pin_1), L502.2
- net RFIO2: now reaches U501.15 (RFO2)
- net RFIO2: now also J501.2 (Pin_2), L501.2
- net at U501.17 (EXT_LIM): now also Q501.2 (G), R502.1
- net AAT_ser: now reaches U501.18 (AAT_A)
- net AAT_ser: now also U502.1 (GND), U503.2 (VT)
- net AAT_par: now reaches U501.19 (AAT_B)
- net AAT_par: now also U504.2 (VT), U505.2 (VT), U506.2 (VT)
- net RFI1: now reaches U501.22 (RFI1)
- net RFI1: now also C531.2, C532.2
- net RFI2: now reaches U501.23 (RFI2)
- net RFI2: now also C533.2, C534.2
- new net: C520.2, C525.1, C528.2, C533.1, R504.1, U503.4 (PORT2), U506.4 (PORT2)
- new net: C525.2, U505.3 (PORT1)
- new net: D502.3 (K), R505.1
- new net: Q501.1 (D), R505.2
- new net: C520.1, C522.2, L501.1, U503.3 (PORT1)
- new net: C521.1, C524.1, C527.1, C531.1, R503.1, U502.4 (PORT2), U504.3 (PORT1)
- new net: C526.2, U506.3 (PORT1)
- new net: C521.2, C523.1, L502.1, U502.3 (PORT1)
- new net: D502.2 (A), R503.2
- new net: D502.1 (A), R504.2
- new net: C524.2, U505.4 (PORT2)
- new net: C526.1, U504.4 (PORT2)
Other:
- note added: "NFC Matching"
- note removed: "Antenna Layout dependent"
- moved on the sheet: R501, U501A, U501D

Commit message: ~layout
Parts:
- added A101: Arduino_UNO_R3, Module:Arduino_UNO_R3, symbol MCU_Module:Arduino_UNO_R3
- L501, L502: footprint (none) -> Inductor_SMD:L_0603_1608Metric_Pad1.05x0.95mm_HandSolder
- U502, U503, U504, U505, U506: footprint LXRW0_MUR -> additional parts:LXRW0_MUR-M
Connections:
- net +3V3: now also A101.4 (3V3)
- net GND: now also A101.29 (GND), A101.6 (GND), A101.7 (GND)
- net NFC_INT: now also A101.9 (A0)
- net NFC_MISO: now also A101.27 (D12)
- net NFC_MOSI: now also A101.26 (D11)
- net NFC_NSS: now also A101.25 (D10)
- net NFC_SCK: now also A101.28 (D13)
- net I2C_Disable renamed I2C_Enable
- no-connect marks 3 -> 25
Other:
- note added: "Antenna"
- note added: "EvalBoard-Connector"
- moved on the sheet: C501, C502, C520, C521, C522, C523, C524, C525, C526, C527, C528, C531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

Commit message: state of pcb ordered
Parts:
- added NT501, NT502: NetTie_2, NetTie:NetTie-2_SMD_Pad0.5mm, symbol Device:NetTie_2
- A101: footprint Module:Arduino_UNO_R3 -> additional parts:Arduino_UNO_R3_no_legend
Connections:
- net GND: now also NT501.2, NT502.2
- net ANT1: now reaches D502.2 (A), R503.2
- net ANT1: now also NT501.1
- net ANT2: now reaches D502.1 (A), R504.2
- net ANT2: now also NT502.1
