File: Hardware/voicemail-box/voicemail-box.kicad_sch (KiCad schematic)
At the start: 8 parts, among them J102 Conn_02x03_Odd_Even, J103 Conn_02x08_Odd_Even, J104 Conn_02x10_Odd_Even, J105 Conn_01x07, J106 Conn_02x10_Odd_Even

Commit message: schema review
Other:
- sheet Pinout CPU ports: added POT1, POT2; removed LED2, LED3
- sheet User Interface ports: added POT1, POT2; removed LED2, LED3
Changed lines of the file:
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@@
-	(wire
-		(pts
-			(xy 50.8 127) (xy 109.22 127)
-		)
-		(stroke
-			(width 0)
-			(type default)
-		)
-	)
 	(wire
 		(pts
@@
 	(wire
 		(pts
+			(xy 50.8 148.59) (xy 109.22 148.59)
+		)
+		(stroke
+			(width 0)
+			(type default)
+		)
+	)
+	(wire
+		(pts
 			(xy 168.91 134.62) (xy 185.42 134.62)
 		)
@@
 	(wire
 		(pts
+			(xy 50.8 146.05) (xy 109.22 146.05)
+		)
+		(stroke
+			(width 0)
+			(type default)
+		)
+	)
+	(wire
+		(pts
 			(xy 227.33 134.62) (xy 217.17 134.62)
 		)
@@
 		(pts
 			(xy 156.21 86.36) (xy 166.37 86.36)
-		)
-		(stroke
-			(width 0)
-			(type default)
-		)
-	)
-	(wire
-		(pts
-			(xy 50.8 129.54) (xy 109.22 129.54)
 		)
 		(stroke
@@
 			)
 		)
-		(pin "LED3" bidirectional
-			(at 50.8 129.54 0)
-			(effects
-				(font
-					(size 1.27 1.27)
-				)
-				(justify right)
-			)
-		)
 		(pin "BTN1" bidirectional
 			(at 50.8 137.16 0)
@@
 			)
 		)
-		(pin "LED2" bidirectional
-			(at 50.8 127 0)
-			(effects
-				(font
-					(size 1.27 1.27)
-				)
-				(justify right)
-			)
-		)
 		(pin "LED1" bidirectional
 			(at 50.8 124.46 0)
@@
 		(pin "BTN2" bidirectional
 			(at 50.8 139.7 0)
+			(effects
+				(font
+					(size 1.27 1.27)
+				)
+				(justify right)
+			)
+		)
+		(pin "POT2" bidirectional
+			(at 50.8 148.59 0)
+			(effects
+				(font
+					(size 1.27 1.27)
+				)
+				(justify right)
+			)
+		)
+		(pin "POT1" bidirectional
+			(at 50.8 146.05 0)
 			(effects
 				(font
@@
 			)
 		)
-		(pin "LED2" bidirectional
-			(at 109.22 127 180)
-			(effects
-				(font
-					(size 1.27 1.27)
-				)
-				(justify left)
-			)
-		)
 		(pin "BTN2" bidirectional
 			(at 109.22 139.7 180)
@@
 			)
 		)
-		(pin "LED3" bidirectional
-			(at 109.22 129.54 180)
-			(effects
-				(font
-					(size 1.27 1.27)
-				)
-				(justify left)
-			)
-		)
 		(pin "LED0" bidirectional
 			(at 109.22 121.92 180)
@@
 			(effects
 				(font
+					(size 1.27 1.27)
+				)
+				(justify left)
+			)
+		)
+		(pin "POT2" bidirectional
+			(at 109.22 148.59 180)
+			(effects
+				(font
+					(size 1.27 1.27)
+				)
+				(justify left)
+			)
+		)
+		(pin "POT1" bidirectional
+			(at 109.22 146.05 180)
+			(effects
+				(font

Commit message: ~layout
Parts:
- removed J105: Conn_01x07, Connector_PinHeader_2.54mm:PinHeader_1x07_P2.54mm_Vertical, symbol Connector_Generic:Conn_01x07
- added J105: Conn_01x08, Connector_PinHeader_2.54mm:PinHeader_1x08_P2.54mm_Vertical, symbol Connector_Generic:Conn_01x08
- added R106, R107: 220R, Resistor_SMD:R_0603_1608Metric_Pad0.98x0.95mm_HandSolder, symbol Device:R
- added RN402: 220R, Resistor_SMD:R_Array_Convex_4x0603, symbol Device:R_Pack04
Connections:
- net GND: now also J105.8 (Pin_8)
- net NFC Breakaway/NFC_INT: now also J105.2 (Pin_2)
- net NFC Breakaway/NFC_MISO: now also J105.6 (Pin_6)
- net NFC Breakaway/NFC_MOSI: now also J105.3 (Pin_3)
- net NFC Breakaway/NFC_NSS: now also J105.5 (Pin_5)
- net NFC Breakaway/NFC_SCK: now also J105.4 (Pin_4)
- net Pinout CPU/MISO: now also RN402.6 (R3.2); no longer J103.6 (Pin_6)
- net Pinout CPU/MOSI: now also RN402.8 (R1.2); no longer J103.2 (Pin_2)
- net Pinout CPU/NSS: now also RN402.7 (R2.2); no longer J103.4 (Pin_4)
- net Pinout CPU/RX: now also R106.2; no longer J103.14 (Pin_14)
- net Pinout CPU/SCK: now also RN402.5 (R4.2); no longer J103.8 (Pin_8)
- net Pinout CPU/TX: now also R107.2; no longer J103.12 (Pin_12)
- net +3.3V renamed +3V3
- net +3V3: now also J105.7 (Pin_7)
- net NFC Breakaway/I2C_Disable renamed NFC Breakaway/I2C_Enable
- net NFC Breakaway/I2C_Enable: now also J105.1 (Pin_1)
- new net: J103.2 (Pin_2), RN402.1 (R1.1)
- new net: J103.4 (Pin_4), RN402.2 (R2.1)
- new net: J103.6 (Pin_6), RN402.3 (R3.1)
- new net: J103.8 (Pin_8), RN402.4 (R4.1)
- new net: J103.14 (Pin_14), R107.1
- new net: J103.12 (Pin_12), R106.1
Other:
- sheet NFC Breakaway ports: added I2C_Enable; removed I2C_Disable
- sheet Pinout CPU ports: added POT0; removed POT2
- sheet User Interface ports: added POT0; removed POT2
- note added: "J103: ------------------ SPI |UART | - set |- open | - set |- open | - set |- open | - set |- open | | | - open |- set | - open |- set | - open |- set |"
- note removed: "J103: ------------------ SPI |I2C | - set |- open | - set |- open | - set |- open | - set |- open | | | - open |- set | - open |- set | - open |- set |"
- moved on the sheet: J102, J103, J104, J106, R101, R102, R103

Commit message: state of pcb ordered
Parts:
- R101, R102: footprint PCM_4ms_Resistor:R_0603 -> Resistor_SMD:R_0603_1608Metric_Pad0.98x0.95mm_HandSolder
Changed lines of the file:
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@@
 			)
 		)
-		(property "Footprint" "PCM_4ms_Resistor:R_0603"
+		(property "Footprint" "Resistor_SMD:R_0603_1608Metric_Pad0.98x0.95mm_HandSolder"
 			(at 154.432 85.09 90)
 			(effects
@@
 			)
 		)
-		(property "Footprint" "PCM_4ms_Resistor:R_0603"
+		(property "Footprint" "Resistor_SMD:R_0603_1608Metric_Pad0.98x0.95mm_HandSolder"
 			(at 164.592 85.09 90)
 			(effects

Commit message: ~ doku
Other:
- note added: "J103: ------------------ SPI |UART | - set |- open | - set |- open | - set |- open | - set |- open | | | - open |- set | - open |- set | - set |- open |"
- note removed: "J103: ------------------ SPI |UART | - set |- open | - set |- open | - set |- open | - set |- open | | | - open |- set | - open |- set | - open |- set |"
Changed lines of the file:
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@@
 		)
 	)
-	(text "J103:\n------------------\nSPI      |UART   |\n- set    |- open |\n- set    |- open |\n- set    |- open |\n- set    |- open |\n         |       |\n- open   |- set  |\n- open   |- set  |\n- open   |- set  |\n"
+	(text "J103:\n------------------\nSPI      |UART   |\n- set    |- open |\n- set    |- open |\n- set    |- open |\n- set    |- open |\n         |       |\n- open   |- set  |\n- open   |- set  |\n- set    |- open |\n"
 		(exclude_from_sim no)
 		(at 88.9 69.342 0)
