File: Hardware/voicemail-box/_autosave-pinout.kicad_sch (KiCad schematic)
At the start: 5 parts, among them CN201 Conn_02x08_Odd_Even

Commit message: + pics ~doku
Other:
- note added: "PA4"
- note added: "PA8 | PA6"
- note added: "PB13 (jumper!)"
- note added: "PB15"
- note added: "PB3"
- note added: "PB5"
- note added: "PB6 | PG14"
- note added: "PB7 | PG9"
- note added: "PD15 | PA7"
- note added: "PE11 | PA2"
- note added: "PE13 | PA1"
- note added: "PE14 | PG12"
- note added: "PG12 | PG11"
- note added: "PG14 | PG13"
- note added: "PG8"
- note added: "PG9 | PG10"
- note removed: "? | PA1"
- note removed: "? | PA6"
- note removed: "? | PA7"
- note removed: "? | PG10"
- note removed: "? | PG12"
- note removed: "? | PG13"
- note removed: "? | PG14"
- note removed: "? | PG9"
- note removed: "?| PA2"
- note removed: "?| PG11"
Changed lines of the file:
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@@
+		)
+	)
+	(text "PB15"
+		(exclude_from_sim no)
+		(at 197.866 31.75 0)
+		(effects
+			(font
+				(face "Courier 10 Pitch")
+				(size 1.27 1.27)
+			)
+			(justify left bottom)
 		)
 	)
@@
 		)
 	)
+	(text "PC7"
+		(exclude_from_sim no)
+		(at 197.866 41.91 0)
+		(effects
+			(font
+				(face "Courier 10 Pitch")
+				(size 1.27 1.27)
+			)
+			(justify left bottom)
+		)
+	)
+	(text "PB4"
+		(exclude_from_sim no)
+		(at 197.866 52.07 0)
+		(effects
+			(font
+				(face "Courier 10 Pitch")
+				(size 1.27 1.27)
+			)
+			(justify left bottom)
+		)
+	)
 	(text "PC1"
 		(exclude_from_sim no)
@@
 		)
 	)
-	(text "?  | PG13"
+	(text "PG14 | PG13"
 		(exclude_from_sim no)
 		(at 235.204 77.47 0)
@@
 		)
 	)
+	(text "PG8"
+		(exclude_from_sim no)
+		(at 102.362 48.26 0)
+		(effects
+			(font
+				(face "Courier 10 Pitch")
+				(size 1.27 1.27)
+			)
+			(justify left bottom)
+		)
+	)
 	(text "PC6"
 		(exclude_from_sim no)
@@
 		)
 	)
+	(text "PA15"
+		(exclude_from_sim no)
+		(at 197.866 39.37 0)
+		(effects
+			(font
+				(face "Courier 10 Pitch")
+				(size 1.27 1.27)
+			)
+			(justify left bottom)
+		)
+	)
 	(text "PC2  | PC5"
 		(exclude_from_sim no)
@@
 		)
 	)
-	(text "?| PA2"
+	(text "PE11 | PA2"
 		(exclude_from_sim no)
 		(at 235.204 69.85 0)
@@
 		)
 	)
+	(text "PA4"
+		(exclude_from_sim no)
+		(at 197.866 49.53 0)
+		(effects
+			(font
+				(face "Courier 10 Pitch")
+				(size 1.27 1.27)
+			)
+			(justify left bottom)
+		)
+	)
+	(text "PC6"
+		(exclude_from_sim no)
+		(at 197.866 29.21 0)
+		(effects
+			(font
+				(face "Courier 10 Pitch")
+				(size 1.27 1.27)
+			)
+			(justify left bottom)
+		)
+	)
 	(text "PC12"
 		(exclude_from_sim no)
@@
 		)
 	)
-	(text "?  | PG14"
+	(text "PB6  | PG14"
 		(exclude_from_sim no)
 		(at 235.204 80.01 0)
@@
 		)
 	)
-	(text "?  | PG12"
+	(text "PB12"
+		(exclude_from_sim no)
+		(at 197.866 36.83 0)
+		(effects
+			(font
+				(face "Courier 10 Pitch")
+				(size 1.27 1.27)
+			)
+			(justify left bottom)
+		)
+	)
+	(text "PE14 | PG12"
 		(exclude_from_sim no)
 		(at 235.204 72.39 0)
@@
 		)
 	)
-	(text "? | PA7"
+	(text "PD15 | PA7"
 		(exclude_from_sim no)
 		(at 233.934 49.53 0)
@@
 		)
 	)
+	(text "H755"
+		(exclude_from_sim no)
+		(at 197.866 26.416 0)
+		(effects
+			(font
+				(face "Courier 10 Pitch")
+				(size 1.27 1.27)
+			)
+			(justify left bottom)
+		)
+	)
+	(text "PB3"
+		(exclude_from_sim no)
+		(at 197.866 46.99 0)
+		(effects
+			(font
+				(face "Courier 10 Pitch")
+				(size 1.27 1.27)
+			)
+			(justify left bottom)
+		)
+	)
 	(text "Orange Marked = Arduino UNO Standard Pinout\nYellow Marked = Nucleo144 Expansion to Arduino Standard"
 		(exclude_from_sim no)
@@
 		)
 	)
-	(text "?| PG11"
+	(text "PG12 | PG11"
 		(exclude_from_sim no)
 		(at 235.204 64.77 0)
@@
 		)
 	)
-	(text "?  | PA1"
+	(text "PE13 | PA1"
 		(exclude_from_sim no)
 		(at 235.204 74.93 0)
@@
 		)
 	)
-	(text "?  | PA6"
+	(text "PA8  | PA6"
 		(exclude_from_sim no)
 		(at 235.204 67.31 0)
@@
 		)
 	)
-	(text "? | PG10"
+	(text "PG9 | PG10"
 		(exclude_from_sim no)
 		(at 233.934 52.07 0)
@@
 		)
 	)
-	(text "? | PG9"
+	(text "PB5"
+		(exclude_from_sim no)
+		(at 197.866 44.45 0)
+		(effects
+			(font
+				(face "Courier 10 Pitch")
+				(size 1.27 1.27)
+			)
+			(justify left bottom)
+		)
+	)
+	(text "PB7  | PG9"
 		(exclude_from_sim no)
 		(at 235.204 82.55 0)
+		(effects
+			(font
+				(face "Courier 10 Pitch")
+				(size 1.27 1.27)
+			)
+			(justify left bottom)
+		)
+	)
+	(text "PB13 (jumper!)"
+		(exclude_from_sim no)
+		(at 193.802 34.29 0)
 		(effects
 			(font
@@
 	(wire
 		(pts
-			(xy 204.47 44.45) (xy 209.55 44.45)
-		)
-		(stroke
-			(width 0)
-			(type default)
-		)
-	)
-	(wire
-		(pts
-			(xy 204.47 34.29) (xy 209.55 34.29)
+			(xy 193.04 44.45) (xy 209.55 44.45)
+		)
+		(stroke
+			(width 0)
+			(type default)
+		)
+	)
+	(wire
+		(pts
+			(xy 193.04 34.29) (xy 209.55 34.29)
 		)
 		(stroke
@@
 	(wire
 		(pts
-			(xy 204.47 36.83) (xy 209.55 36.83)
+			(xy 193.04 36.83) (xy 209.55 36.83)
 		)
 		(stroke
@@
 	(wire
 		(pts
-			(xy 204.47 46.99) (xy 209.55 46.99)
+			(xy 193.04 46.99) (xy 209.55 46.99)
 		)
 		(stroke
@@
 	(wire
 		(pts
-			(xy 204.47 31.75) (xy 209.55 31.75)
+			(xy 193.04 31.75) (xy 209.55 31.75)
 		)
 		(stroke
@@
 	(wire
 		(pts
-			(xy 204.47 29.21) (xy 209.55 29.21)
+			(xy 193.04 29.21) (xy 209.55 29.21)
 		)
 		(stroke
@@
 	(wire
 		(pts
-			(xy 204.47 52.07) (xy 209.55 52.07)
+			(xy 193.04 52.07) (xy 209.55 52.07)
 		)
 		(stroke
@@
 	(wire
 		(pts
-			(xy 204.47 49.53) (xy 209.55 49.53)
+			(xy 193.04 49.53) (xy 209.55 49.53)
 		)
 		(stroke
@@
 	(hierarchical_label "I2S_MCLK"
 		(shape bidirectional)
-		(at 204.47 29.21 180)
+		(at 193.04 29.21 180)
 		(effects
 			(font
@@
 	(hierarchical_label "SPI2_NSS"
 		(shape bidirectional)
-		(at 204.47 49.53 180)
+		(at 193.04 49.53 180)
 		(effects
 			(font
@@
 	(hierarchical_label "SPI2_SCK"
 		(shape bidirectional)
-		(at 204.47 46.99 180)
+		(at 193.04 46.99 180)
 		(effects
 			(font
@@
 	(hierarchical_label "I2S_BCLK"
 		(shape bidirectional)
-		(at 204.47 34.29 180)
+		(at 193.04 34.29 180)
 		(effects
 			(font
@@
 	(hierarchical_label "I2S_SDA"
 		(shape bidirectional)
-		(at 204.47 31.75 180)
+		(at 193.04 31.75 180)
 		(effects
 			(font
@@
 	(hierarchical_label "I2S_SDA_ext"
 		(shape bidirectional)
-		(at 204.47 52.07 180)
+		(at 193.04 52.07 180)
 		(effects
 			(font
@@
 	(hierarchical_label "SPI2_MOSI"
 		(shape bidirectional)
-		(at 204.47 44.45 180)
+		(at 193.04 44.45 180)
 		(effects
 			(font
@@
 	(hierarchical_label "I2S_WCLK"
 		(shape bidirectional)
-		(at 204.47 36.83 180)
-		(effects
-			(font
+		(at 193.04 36.83 180)
+		(effects
+			(font
