File: Hardware/PCB/powersupply.kicad_sch (KiCad schematic)
At the start: 12 parts, among them J701 USB_C_Receptacle_PowerOnly_6P, U701 R-78B3.3-2.0, U702 TC2015-1.8VxCTTR

Commit message: ~ hw-files update
Parts:
- J701: Part Number (none) -> 10164359-00011LF
Changed lines of the file:
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@@
+			)
+		)
+		(property "Part Number" "10164359-00011LF"
+			(at 69.85 85.09 0)
+			(effects
+				(font
+					(size 1.27 1.27)
+				)
+				(hide yes)
 			)
 		)

Commit message: ~fixes on schematic and pcb ~prep for final output generation
Parts:
- C805, C807, C809: Manufacturer (none) -> Kemet; Part Number (none) -> C0603C104K5RACTUCT
- C806, C808: Manufacturer (none) -> Kemet; Part Number (none) -> C0603C106M9PAC7411
- C810: Manufacturer (none) -> Kemet; Part Number (none) -> C0603C102K5RACTUCT
- J701: Manufacturer (none) -> Amphenol ICC (FCI)
- R701, R702: Manufacturer (none) -> Yageo; Part Number (none) -> RC0603FR-075K1L
- U701: Manufacturer (none) -> Recom Power; Part Number (none) -> R-78K3.3-2.0
- U702: Manufacturer (none) -> Microchip Technology; Part Number (none) -> MIC5259-1.8YD5-TR
Changed lines of the file:
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@@
+			)
+		)
+		(property "Manufacturer" "Microchip Technology"
+			(at 195.58 80.01 0)
+			(effects
+				(font
+					(size 1.27 1.27)
+				)
+				(hide yes)
+			)
+		)
+		(property "Part Number" "MIC5259-1.8YD5-TR"
+			(at 195.58 80.01 0)
+			(effects
+				(font
+					(size 1.27 1.27)
+				)
+				(hide yes)
 			)
 		)
@@
 			)
 		)
+		(property "Manufacturer" "Kemet"
+			(at 176.53 90.17 0)
+			(effects
+				(font
+					(size 1.27 1.27)
+				)
+				(hide yes)
+			)
+		)
+		(property "Part Number" "C0603C106M9PAC7411"
+			(at 176.53 90.17 0)
+			(effects
+				(font
+					(size 1.27 1.27)
+				)
+				(hide yes)
+			)
+		)
 		(pin "2"
 		)
@@
 			)
 		)
+		(property "Manufacturer" "Kemet"
+			(at 125.73 90.17 0)
+			(effects
+				(font
+					(size 1.27 1.27)
+				)
+				(hide yes)
+			)
+		)
+		(property "Part Number" "C0603C104K5RACTUCT"
+			(at 125.73 90.17 0)
+			(effects
+				(font
+					(size 1.27 1.27)
+				)
+				(hide yes)
+			)
+		)
 		(pin "2"
 		)
@@
 			)
 		)
+		(property "Manufacturer" "Yageo"
+			(at 88.9 100.33 0)
+			(effects
+				(font
+					(size 1.27 1.27)
+				)
+				(hide yes)
+			)
+		)
+		(property "Part Number" "RC0603FR-075K1L"
+			(at 88.9 100.33 0)
+			(effects
+				(font
+					(size 1.27 1.27)
+				)
+				(hide yes)
+			)
+		)
 		(pin "2"
 		)
@@
 			)
 		)
+		(property "Manufacturer" "Amphenol ICC (FCI)"
+			(at 69.85 85.09 0)
+			(effects
+				(font
+					(size 1.27 1.27)
+				)
+				(hide yes)
+			)
+		)
 		(pin "A12"
 		)
@@
 			)
 		)
+		(property "Manufacturer" "Kemet"
+			(at 163.83 90.17 0)
+			(effects
+				(font
+					(size 1.27 1.27)
+				)
+				(hide yes)
+			)
+		)
+		(property "Part Number" "C0603C104K5RACTUCT"
+			(at 163.83 90.17 0)
+			(effects
+				(font
+					(size 1.27 1.27)
+				)
+				(hide yes)
+			)
+		)
 		(pin "2"
 		)
@@
 			)
 		)
+		(property "Manufacturer" "Kemet"
+			(at 138.43 90.17 0)
+			(effects
+				(font
+					(size 1.27 1.27)
+				)
+				(hide yes)
+			)
+		)
+		(property "Part Number" "C0603C106M9PAC7411"
+			(at 138.43 90.17 0)
+			(effects
+				(font
+					(size 1.27 1.27)
+				)
+				(hide yes)
+			)
+		)
 		(pin "2"
 		)
@@
 		)
 		(property "Description" "Resistor"
+			(at 99.06 100.33 0)
+			(effects
+				(font
+					(size 1.27 1.27)
+				)
+				(hide yes)
+			)
+		)
+		(property "Manufacturer" "Yageo"
+			(at 99.06 100.33 0)
+			(effects
+				(font
+					(size 1.27 1.27)
+				)
+				(hide yes)
+			)
+		)
+		(property "Part Number" "RC0603FR-075K1L"
 			(at 99.06 100.33 0)
 			(effects
@@
 			)
 		)
+		(property "Manufacturer" "Recom Power"
+			(at 149.86 77.47 0)
+			(effects
+				(font
+					(size 1.27 1.27)
+				)
+				(hide yes)
+			)
+		)
+		(property "Part Number" "R-78K3.3-2.0"
+			(at 149.86 77.47 0)
+			(effects
+				(font
+					(size 1.27 1.27)
+				)
+				(hide yes)
+			)
+		)
 		(pin "3"
 		)
@@
 			)
 		)
+		(property "Manufacturer" "Kemet"
+			(at 209.55 90.17 0)
+			(effects
+				(font
+					(size 1.27 1.27)
+				)
+				(hide yes)
+			)
+		)
+		(property "Part Number" "C0603C104K5RACTUCT"
+			(at 209.55 90.17 0)
+			(effects
+				(font
+					(size 1.27 1.27)
+				)
+				(hide yes)
+			)
+		)
 		(pin "2"
 		)
@@
 			(at 107.95 90.17 0)
 			(effects
+				(font
+					(size 1.27 1.27)
+				)
+				(hide yes)
+			)
+		)
+		(property "Manufacturer" "Kemet"
+			(at 107.95 90.17 0)
+			(effects
+				(font
+					(size 1.27 1.27)
+				)
+				(hide yes)
+			)
+		)
+		(property "Part Number" "C0603C102K5RACTUCT"
+			(at 107.95 90.17 0)
+			(effects

Commit message: ~ board 3D files improved ~ bom output prep
Parts:
- J701: footprint Connector_USB:USB_C_Receptacle_HRO_TYPE-C-31-M-17 -> additional parts:USB_C_Receptacle_HRO_TYPE-C-31-M-17
Changed lines of the file:
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@@
 			)
 		)
-		(property "Footprint" "Connector_USB:USB_C_Receptacle_HRO_TYPE-C-31-M-17"
+		(property "Footprint" "additional parts:USB_C_Receptacle_HRO_TYPE-C-31-M-17"
 			(at 73.66 82.55 0)
 			(effects
