File: Hardware/PCB/userinterface.kicad_sch (KiCad schematic)
At the start: 29 parts, among them J801 Conn_01x08, J802 Conn_02x03_Odd_Even, J803 Conn_02x03_Odd_Even, SW801 Push_Button, SW802 Push_Button, SW803 Push_Button, SW804 Push_Button, U801 74LS07

Commit message: ~ hw-files update
Parts:
- LED801: Manufacturer Kingbright -> (none); Part Number AP1608SRCPRV -> LTST-C190KFKT
- LED804: Manufacturer Inolux -> (none); Part Number IN-S63AT5G -> LTST-C190GKT
Changed lines of the file:
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@@
 			)
 		)
-		(property "Manufacturer" "Kingbright"
+		(property "Manufacturer" ""
 			(at 165.608 31.75 0)
 			(effects
@@
 			)
 		)
-		(property "Part Number" "AP1608SRCPRV"
+		(property "Part Number" "LTST-C190KFKT"
 			(at 167.132 31.75 0)
 			(effects
@@
 			)
 		)
-		(property "Manufacturer" "Inolux"
+		(property "Manufacturer" ""
 			(at 151.638 31.75 0)
 			(effects
@@
 			)
 		)
-		(property "Part Number" "IN-S63AT5G"
+		(property "Part Number" "LTST-C190GKT"
 			(at 153.162 31.75 0)
 			(effects

Commit message: ~fixes on schematic and pcb ~prep for final output generation
Parts:
- C811, C812, C813, C814, C815: Manufacturer (none) -> Kemet; Part Number (none) -> C0603C104K5RACTUCT
- J802, J803: footprint Connector_PinSocket_2.54mm:PinSocket_2x03_P2.54mm_Vertical -> Connector_PinHeader_2.54mm:PinHeader_2x03_P2.54mm_Vertical; Manufacturer (none) -> Würth Elektronik; Part Number (none) -> 61300621121
- LED801, LED804: Manufacturer (none) -> Lite-On Inc.
- R801, R802: Manufacturer (none) -> Yageo; Part Number (none) -> RC0603FR-071K2L
- R805, R806, R807, R808, R809, R810, R811, R812, R813, R814: Manufacturer (none) -> Yageo; Part Number (none) -> RC0603FR-074K7L
- RV801, RV802: Manufacturer (none) -> Alps Alpine; Part Number (none) -> RK1631110U2A
- SW801, SW802, SW803, SW804: Manufacturer (none) -> Same Sky (Formerly CUI Devices); Part Number (none) -> TS02-66-70-BK-100-SCR-D
- U801: Manufacturer (none) -> Texas Instruments; Part Number (none) -> SN74LS07DR
Connections:
- net +3V3: now also J802.1 (Pin_1), J803.1 (Pin_1); no longer J802.2 (Pin_2), J803.2 (Pin_2)
- net GND: now also J802.5 (Pin_5), J803.5 (Pin_5); no longer J802.6 (Pin_6), J803.6 (Pin_6)
- net POT0: now also J802.4 (Pin_4); no longer J802.3 (Pin_3)
- net POT1: now also J803.4 (Pin_4); no longer J803.3 (Pin_3)
- net ext_Poti0: now also J802.3 (Pin_3), J802.6 (Pin_6); no longer J802.4 (Pin_4), J802.5 (Pin_5)
- net ext_Poti1: now also J803.3 (Pin_3), J803.6 (Pin_6); no longer J803.4 (Pin_4), J803.5 (Pin_5)
- net at RV801.2: now also J802.2 (Pin_2); no longer J802.1 (Pin_1)
- net at RV802.2: now also J803.2 (Pin_2); no longer J803.1 (Pin_1)

Commit message: ~ board 3D files improved ~ bom output prep
Parts:
- J801: Manufacturer (none) -> Würth Elektronik; Part Number (none) -> 61300811121
Changed lines of the file:
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@@
+			)
+		)
+		(property "Manufacturer" "Würth Elektronik"
+			(at 67.31 113.03 0)
+			(effects
+				(font
+					(size 1.27 1.27)
+				)
+				(hide yes)
+			)
+		)
+		(property "Part Number" "61300811121"
+			(at 67.31 113.03 0)
+			(effects
+				(font
+					(size 1.27 1.27)
+				)
+				(hide yes)
 			)
 		)
