File: Hardware/PCB/voicemail-box.kicad_sch (KiCad schematic)
At the start: 11 parts, among them J102 Conn_02x03_Odd_Even, J103 Conn_02x08_Odd_Even, J104 Conn_02x10_Odd_Even, J105 Conn_01x08, J106 Conn_02x10_Odd_Even

Commit message: ~fixes on schematic and pcb ~prep for final output generation
Parts:
- J102: Manufacturer (none) -> Würth Elektronik; Part Number (none) -> 61300621121
- J103: Manufacturer (none) -> Würth Elektronik; Part Number (none) -> 61301621121
- J104, J106: Manufacturer (none) -> Molex; Part Number (none) -> 0901310770
- R101, R102: Manufacturer (none) -> Yageo; Part Number (none) -> RC0603FR-074K7L
- R103: footprint PCM_4ms_Resistor:R_0603 -> Resistor_SMD:R_0603_1608Metric_Pad0.98x0.95mm_HandSolder; Manufacturer (none) -> Yageo; Part Number (none) -> RC0603FR-074K7L
- R106, R107: Manufacturer (none) -> Yageo; Part Number (none) -> RC0603FR-07220RL
- RN402: Manufacturer (none) -> Panasonic Electronic Components; Part Number (none) -> EXB-38V221JV
Changed lines of the file:
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@@
+			)
+		)
+		(property "Manufacturer" "Panasonic Electronic Components"
+			(at 91.44 35.56 0)
+			(effects
+				(font
+					(size 1.27 1.27)
+				)
+				(hide yes)
+			)
+		)
+		(property "Part Number" "EXB-38V221JV"
+			(at 91.44 35.56 0)
+			(effects
+				(font
+					(size 1.27 1.27)
+				)
+				(hide yes)
 			)
 		)
@@
 			)
 		)
+		(property "Manufacturer" "Yageo"
+			(at 156.21 85.09 0)
+			(effects
+				(font
+					(size 1.27 1.27)
+				)
+				(hide yes)
+			)
+		)
+		(property "Part Number" "RC0603FR-074K7L"
+			(at 156.21 85.09 0)
+			(effects
+				(font
+					(size 1.27 1.27)
+				)
+				(hide yes)
+			)
+		)
 		(pin "1"
 		)
@@
 			)
 		)
+		(property "Manufacturer" "Yageo"
+			(at 91.44 49.53 90)
+			(effects
+				(font
+					(size 1.27 1.27)
+				)
+				(hide yes)
+			)
+		)
+		(property "Part Number" "RC0603FR-07220RL"
+			(at 91.44 49.53 90)
+			(effects
+				(font
+					(size 1.27 1.27)
+				)
+				(hide yes)
+			)
+		)
 		(pin "1"
 		)
@@
 		)
 		(property "Description" "Generic connector, double row, 02x10, odd/even pin numbering scheme (row 1 odd numbers, row 2 even numbers), script generated (kicad-library-utils/schlib/autogen/connector/)"
+			(at 161.29 120.65 0)
+			(effects
+				(font
+					(size 1.27 1.27)
+				)
+				(hide yes)
+			)
+		)
+		(property "Manufacturer" "Molex"
+			(at 161.29 120.65 0)
+			(effects
+				(font
+					(size 1.27 1.27)
+				)
+				(hide yes)
+			)
+		)
+		(property "Part Number" "0901310770"
 			(at 161.29 120.65 0)
 			(effects
@@
 			)
 		)
-		(property "Footprint" "PCM_4ms_Resistor:R_0603"
+		(property "Footprint" "Resistor_SMD:R_0603_1608Metric_Pad0.98x0.95mm_HandSolder"
 			(at 66.802 62.23 90)
 			(effects
@@
 		)
 		(property "Description" "Resistor"
+			(at 68.58 62.23 0)
+			(effects
+				(font
+					(size 1.27 1.27)
+				)
+				(hide yes)
+			)
+		)
+		(property "Manufacturer" "Yageo"
+			(at 68.58 62.23 0)
+			(effects
+				(font
+					(size 1.27 1.27)
+				)
+				(hide yes)
+			)
+		)
+		(property "Part Number" "RC0603FR-074K7L"
 			(at 68.58 62.23 0)
 			(effects
@@
 			)
 		)
+		(property "Manufacturer" "Yageo"
+			(at 166.37 85.09 0)
+			(effects
+				(font
+					(size 1.27 1.27)
+				)
+				(hide yes)
+			)
+		)
+		(property "Part Number" "RC0603FR-074K7L"
+			(at 166.37 85.09 0)
+			(effects
+				(font
+					(size 1.27 1.27)
+				)
+				(hide yes)
+			)
+		)
 		(pin "1"
 		)
@@
 			)
 		)
+		(property "Manufacturer" "Würth Elektronik"
+			(at 190.5 102.87 90)
+			(effects
+				(font
+					(size 1.27 1.27)
+				)
+				(hide yes)
+			)
+		)
+		(property "Part Number" "61300621121"
+			(at 190.5 102.87 90)
+			(effects
+				(font
+					(size 1.27 1.27)
+				)
+				(hide yes)
+			)
+		)
 		(pin "3"
 		)
@@
 		(property "Description" "Resistor"
 			(at 91.44 43.18 0)
+			(effects
+				(font
+					(size 1.27 1.27)
+				)
+				(hide yes)
+			)
+		)
+		(property "Manufacturer" "Yageo"
+			(at 91.44 43.18 90)
+			(effects
+				(font
+					(size 1.27 1.27)
+				)
+				(hide yes)
+			)
+		)
+		(property "Part Number" "RC0603FR-07220RL"
+			(at 91.44 43.18 90)
 			(effects
 				(font
@@
 			)
 		)
+		(property "Manufacturer" "Molex"
+			(at 172.72 54.61 0)
+			(effects
+				(font
+					(size 1.27 1.27)
+				)
+				(hide yes)
+			)
+		)
+		(property "Part Number" "0901310770"
+			(at 172.72 54.61 0)
+			(effects
+				(font
+					(size 1.27 1.27)
+				)
+				(hide yes)
+			)
+		)
 		(pin "19"
 		)
@@
 			(at 73.66 38.1 0)
 			(effects
+				(font
+					(size 1.27 1.27)
+				)
+				(hide yes)
+			)
+		)
+		(property "Manufacturer" "Würth Elektronik"
+			(at 73.66 38.1 0)
+			(effects
+				(font
+					(size 1.27 1.27)
+				)
+				(hide yes)
+			)
+		)
+		(property "Part Number" "61301621121"
+			(at 73.66 38.1 0)
+			(effects

Commit message: ~ board 3D files improved ~ bom output prep
Parts:
- J105: Manufacturer (none) -> Würth Elektronik; Part Number (none) -> 61300811121
Changed lines of the file:
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@@
+			)
+		)
+		(property "Manufacturer" "Würth Elektronik"
+			(at 232.41 128.27 0)
+			(effects
+				(font
+					(size 1.27 1.27)
+				)
+				(hide yes)
+			)
+		)
+		(property "Part Number" "61300811121"
+			(at 232.41 128.27 0)
+			(effects
+				(font
+					(size 1.27 1.27)
+				)
+				(hide yes)
 			)
 		)
