File: Hardware/PCB/nucleo144_ext.kicad_sch (KiCad schematic)
At the start: 5 parts, among them J401 Micro_SD_Card_Det1

Commit message: ~ hw-files update
Parts:
- J401: Part Number (none) -> DM3AT-SF-PEJM5
Changed lines of the file:
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@@
+			)
+		)
+		(property "Part Number" "DM3AT-SF-PEJM5"
+			(at 123.19 52.07 0)
+			(effects
+				(font
+					(size 1.27 1.27)
+				)
+				(hide yes)
 			)
 		)

Commit message: ~fixes on schematic and pcb ~prep for final output generation
Parts:
- C401: Manufacturer (none) -> Kemet; Part Number (none) -> C0805C104K5RACTU
- J401: Manufacturer (none) -> Hirose Electric Co Ltd
- R506, R507: Manufacturer (none) -> Yageo; Part Number (none) -> RC0603FR-0710KL
- RN401: Manufacturer (none) -> Panasonic Electronic Components; Part Number (none) -> EXB-38V103JV
Changed lines of the file:
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@@
+			)
+		)
+		(property "Manufacturer" "Kemet"
+			(at 147.32 59.69 0)
+			(effects
+				(font
+					(size 1.27 1.27)
+				)
+				(hide yes)
+			)
+		)
+		(property "Part Number" "C0805C104K5RACTU"
+			(at 147.32 59.69 0)
+			(effects
+				(font
+					(size 1.27 1.27)
+				)
+				(hide yes)
 			)
 		)
@@
 		)
 		(property "Description" "4 resistor network, parallel topology"
+			(at 54.61 39.37 0)
+			(effects
+				(font
+					(size 1.27 1.27)
+				)
+				(hide yes)
+			)
+		)
+		(property "Manufacturer" "Panasonic Electronic Components"
+			(at 54.61 39.37 0)
+			(effects
+				(font
+					(size 1.27 1.27)
+				)
+				(hide yes)
+			)
+		)
+		(property "Part Number" "EXB-38V103JV"
 			(at 54.61 39.37 0)
 			(effects
@@
 		)
 		(property "Description" "Resistor"
+			(at 39.37 39.37 0)
+			(effects
+				(font
+					(size 1.27 1.27)
+				)
+				(hide yes)
+			)
+		)
+		(property "Manufacturer" "Yageo"
+			(at 39.37 39.37 0)
+			(effects
+				(font
+					(size 1.27 1.27)
+				)
+				(hide yes)
+			)
+		)
+		(property "Part Number" "RC0603FR-0710KL"
 			(at 39.37 39.37 0)
 			(effects
@@
 			)
 		)
+		(property "Manufacturer" "Hirose Electric Co Ltd"
+			(at 123.19 52.07 0)
+			(effects
+				(font
+					(size 1.27 1.27)
+				)
+				(hide yes)
+			)
+		)
 		(pin "10"
 		)
@@
 			(at 48.26 39.37 0)
 			(effects
+				(font
+					(size 1.27 1.27)
+				)
+				(hide yes)
+			)
+		)
+		(property "Manufacturer" "Yageo"
+			(at 48.26 39.37 0)
+			(effects
+				(font
+					(size 1.27 1.27)
+				)
+				(hide yes)
+			)
+		)
+		(property "Part Number" "RC0603FR-0710KL"
+			(at 48.26 39.37 0)
+			(effects

Commit message: finaly working variants
Parts:
- R506, R507: Var (none) -> Assembly Full(+!) Partial(+!)
Changed lines of the file:
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@@
+			)
+		)
+		(property "Var" "Assembly Full(+!) Partial(+!)"
+			(at 39.37 39.37 0)
+			(effects
+				(font
+					(size 1.27 1.27)
+				)
+				(hide yes)
 			)
 		)
@@
 			(at 48.26 39.37 0)
 			(effects
+				(font
+					(size 1.27 1.27)
+				)
+				(hide yes)
+			)
+		)
+		(property "Var" "Assembly Full(+!) Partial(+!)"
+			(at 48.26 39.37 0)
+			(effects
