File: Hardware/PCB/NFC_breakaway.kicad_sch (KiCad schematic)
At the start: 52 parts, among them J501 Conn_01x02, Q501 NX3008NBK, U501 ST25R3916B, U502 LXRW0YV600-054, U503 LXRW0YV600-054, U504 LXRW0YV600-054, U505 LXRW0YV600-054, U506 LXRW0YV600-054, Y501 27.12Mhz

Commit message: ~ hw-files update
Parts:
- C501, C502, C531: Manufacturer (none) -> Kemet; Part Number (none) -> C0603C100K5GACTU
- C505, C507, C509, C513, C515, C517, C519: Manufacturer (none) -> Kemet; Part Number (none) -> C0603C225K4PACTU
- C511: Manufacturer (none) -> Kemet; Part Number (none) -> C0603C105K4RACTU
- C514: Manufacturer (none) -> Kemet; Part Number (none) -> C0603C223K1RACTU
- C520, C521: Manufacturer (none) -> Kemet; Part Number (none) -> C0603C101J5GACTU
- C522, C523: Manufacturer (none) -> Kemet; Part Number (none) -> C0603C681K5RACTU
- C524, C525, C526: Manufacturer (none) -> Kemet; Part Number (none) -> C0603C470K5GACTU
- C527, C528: Manufacturer (none) -> Kemet; Part Number (none) -> C0603C560M3HACTU
- C532, C534: Manufacturer (none) -> Kemet; Part Number (none) -> C0603C181J5GACTU
- C533: Digikey (none) -> 399-C0603C100K5GACTUCT-ND; Manufacturer (none) -> Kemet; Part Number (none) -> C0603C100K5GACTU
- D502: Part Number (none) -> BAV70W-7-F
- L501, L502: Manufacturer (none) -> Murata; Part Number (none) -> LQW18ANR27J00D

Commit message: ~fixes on schematic and pcb ~prep for final output generation
Parts:
- C501, C502, C505, C507, C509, C511, C513, C514, C515, C517, C519, C520, C521, C522, C523, C524, C525, C526, C527, C528, C531, C532, C533, C534, L501, L502: now not fitted
- C503, C504, C506, C508, C510, C512, C516, C518: Manufacturer (none) -> Kemet; Part Number (none) -> C0603C103K5RACTU; now not fitted
- D502: Manufacturer (none) -> Diodes Incorporated
- J501: Manufacturer (none) -> Harwin Inc.; Part Number (none) -> M50-3532042; now not fitted
- Q501: Manufacturer (none) -> Nexperia USA Inc.; Part Number (none) -> NX3008NBKW,115; now not fitted
- R501: Manufacturer (none) -> Yageo; Part Number (none) -> RC0603FR-0710KL; now not fitted
- R502: Manufacturer (none) -> Yageo; Part Number (none) -> RC0603FR-0747KL; now not fitted
- R503, R504: Manufacturer (none) -> Yageo; Part Number (none) -> RC0603FR-072K4L; now not fitted
- R505: Manufacturer (none) -> Yageo; Part Number (none) -> RC0805FR-07100RL; now not fitted
- U501: Manufacturer (none) -> STMicroelectronics; Part Number (none) -> ST25R3916B-AQET; now not fitted
- U502, U503, U504, U505, U506: Manufacturer (none) -> Murata Electronics; Part Number (none) -> LXRW0YV600-054; now not fitted
- Y501: Manufacturer (none) -> EPSON; Part Number (none) -> FA-118T 27.1200MD50Z-K3; now not fitted

Commit message: ~ board 3D files improved ~ bom output prep
Parts:
- A101: now not fitted
- C501, C502, C503, C504, C505, C506, C507, C508, C509, C510, C511, C512, C513, C514, C515, C516, C517, C518, C519, C520, C521, C522, C523, C524, C525, C526, C527, C528, C531, C532, C533, C534, J501, L501, L502, Q501, R501, R502, R503, R504, R505, U502, U503, U504, U505, U506, Y501: now fitted
- U501: footprint Package_DFN_QFN:UFQFPN-32-1EP_5x5mm_P0.5mm_EP3.5x3.5mm -> additional parts:UFQFPN-32-1EP_5x5mm_P0.5mm_EP3.5x3.5mm; now fitted
Changed lines of the file:
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@@
 		(in_bom yes)
 		(on_board yes)
-		(dnp yes)
+		(dnp no)
 		(property "Reference" "U501"
 			(at 135.636 165.1 0)
@@
 			)
 		)
-		(property "Footprint" "Package_DFN_QFN:UFQFPN-32-1EP_5x5mm_P0.5mm_EP3.5x3.5mm"
+		(property "Footprint" "additional parts:UFQFPN-32-1EP_5x5mm_P0.5mm_EP3.5x3.5mm"
 			(at 137.16 166.37 0)
 			(effects
@@
 		(in_bom yes)
 		(on_board yes)
-		(dnp yes)
+		(dnp no)
 		(fields_autoplaced yes)
 		(property "Reference" "R502"
@@
 		(in_bom yes)
 		(on_board yes)
-		(dnp yes)
+		(dnp no)
 		(fields_autoplaced yes)
 		(property "Reference" "C525"
@@
 		(in_bom yes)
 		(on_board yes)
-		(dnp yes)
+		(dnp no)
 		(fields_autoplaced yes)
 		(property "Reference" "R505"
@@
 		(in_bom yes)
 		(on_board yes)
-		(dnp yes)
+		(dnp no)
 		(fields_autoplaced yes)
 		(property "Reference" "C522"
@@
 		(in_bom yes)
 		(on_board yes)
-		(dnp yes)
+		(dnp no)
 		(property "Reference" "C501"
 			(at 256.54 95.25 0)
@@
 		(in_bom yes)
 		(on_board yes)
-		(dnp yes)
+		(dnp no)
 		(property "Reference" "Q501"
 			(at 239.776 86.868 0)
@@
 		(in_bom yes)
 		(on_board yes)
-		(dnp yes)
+		(dnp no)
 		(property "Reference" "C502"
 			(at 279.4 95.25 0)
@@
 		(in_bom yes)
 		(on_board yes)
-		(dnp yes)
+		(dnp no)
 		(property "Reference" "U501"
 			(at 263.906 61.976 90)
@@
 			)
 		)
-		(property "Footprint" "Package_DFN_QFN:UFQFPN-32-1EP_5x5mm_P0.5mm_EP3.5x3.5mm"
+		(property "Footprint" "additional parts:UFQFPN-32-1EP_5x5mm_P0.5mm_EP3.5x3.5mm"
 			(at 260.35 69.85 0)
 			(effects
@@
 		(in_bom yes)
 		(on_board yes)
-		(dnp yes)
+		(dnp no)
 		(property "Reference" "C513"
 			(at 210.82 138.43 0)
@@
 		(in_bom yes)
 		(on_board yes)
-		(dnp yes)
+		(dnp no)
 		(property "Reference" "C507"
 			(at 115.57 138.43 0)
@@
 		(in_bom yes)
 		(on_board yes)
-		(dnp yes)
+		(dnp no)
 		(fields_autoplaced yes)
 		(property "Reference" "C527"
@@
 		(in_bom yes)
 		(on_board yes)
-		(dnp yes)
+		(dnp no)
 		(property "Reference" "U506"
 			(at 180.34 59.69 0)
@@
 		(in_bom yes)
 		(on_board yes)
-		(dnp yes)
+		(dnp no)
 		(fields_autoplaced yes)
 		(property "Reference" "C521"
@@
 		(in_bom yes)
 		(on_board yes)
-		(dnp yes)
+		(dnp no)
 		(fields_autoplaced yes)
 		(property "Reference" "Y501"
@@
 		(in_bom yes)
 		(on_board yes)
-		(dnp yes)
+		(dnp no)
 		(fields_autoplaced yes)
 		(property "Reference" "R503"
@@
 		(in_bom yes)
 		(on_board yes)
-		(dnp yes)
+		(dnp no)
 		(property "Reference" "C505"
 			(at 95.25 138.43 0)
@@
 		(in_bom yes)
 		(on_board yes)
-		(dnp yes)
+		(dnp no)
 		(property "Reference" "C532"
 			(at 95.25 14.732 90)
@@
 		(in_bom yes)
 		(on_board yes)
-		(dnp yes)
+		(dnp no)
 		(property "Reference" "C518"
 			(at 261.62 138.43 0)
@@
 		(in_bom yes)
 		(on_board yes)
-		(dnp yes)
+		(dnp no)
 		(property "Reference" "L502"
 			(at 96.52 41.402 90)
@@
 		(in_bom yes)
 		(on_board yes)
-		(dnp yes)
+		(dnp no)
 		(fields_autoplaced yes)
 		(property "Reference" "C528"
@@
 		(in_bom yes)
 		(on_board yes)
-		(dnp yes)
+		(dnp no)
 		(property "Reference" "U501"
 			(at 13.716 60.96 0)
@@
 			)
 		)
-		(property "Footprint" "Package_DFN_QFN:UFQFPN-32-1EP_5x5mm_P0.5mm_EP3.5x3.5mm"
+		(property "Footprint" "additional parts:UFQFPN-32-1EP_5x5mm_P0.5mm_EP3.5x3.5mm"
 			(at 15.24 62.23 0)
 			(effects
@@
 		(in_bom yes)
 		(on_board yes)
-		(dnp yes)
+		(dnp no)
 		(fields_autoplaced yes)
 		(property "Reference" "J501"
@@
 		(in_bom yes)
 		(on_board yes)
-		(dnp yes)
+		(dnp no)
 		(property "Reference" "C511"
 			(at 156.21 138.43 0)
@@
 		(in_bom yes)
 		(on_board yes)
-		(dnp yes)
+		(dnp no)
 		(fields_autoplaced yes)
 		(property "Reference" "C524"
@@
 		(in_bom yes)
 		(on_board yes)
-		(dnp yes)
+		(dnp no)
 		(property "Reference" "C503"
 			(at 74.93 138.43 0)
@@
 		(in_bom yes)
 		(on_board yes)
-		(dnp yes)
+		(dnp no)
 		(property "Reference" "L501"
 			(at 96.52 70.612 90)
@@
 		(in_bom yes)
 		(on_board yes)
-		(dnp yes)
+		(dnp no)
 		(property "Reference" "C509"
 			(at 135.89 138.43 0)
@@
 		(in_bom yes)
 		(on_board yes)
-		(dnp yes)
+		(dnp no)
 		(property "Reference" "C516"
 			(at 241.3 138.43 0)
@@
 		(in_bom yes)
 		(on_board yes)
-		(dnp no)
+		(dnp yes)
 		(fields_autoplaced yes)
 		(property "Reference" "A101"
@@
 		(in_bom yes)
 		(on_board yes)
-		(dnp yes)
+		(dnp no)
 		(property "Reference" "C504"
 			(at 85.09 138.43 0)
@@
 		(in_bom yes)
 		(on_board yes)
-		(dnp yes)
+		(dnp no)
 		(property "Reference" "C514"
 			(at 220.98 138.43 0)
@@
 		(in_bom yes)
 		(on_board yes)
-		(dnp yes)
+		(dnp no)
 		(fields_autoplaced yes)
 		(property "Reference" "C531"
@@
 		(in_bom yes)
 		(on_board yes)
-		(dnp yes)
+		(dnp no)
 		(property "Reference" "C515"
 			(at 231.14 138.43 0)
@@
 		(in_bom yes)
 		(on_board yes)
-		(dnp yes)
+		(dnp no)
 		(property "Reference" "U502"
 			(at 60.96 46.99 0)
@@
 		(in_bom yes)
 		(on_board yes)
-		(dnp yes)
+		(dnp no)
 		(property "Reference" "U501"
 			(at 167.894 119.38 0)
@@
 			)
 		)
-		(property "Footprint" "Package_DFN_QFN:UFQFPN-32-1EP_5x5mm_P0.5mm_EP3.5x3.5mm"
+		(property "Footprint" "additional parts:UFQFPN-32-1EP_5x5mm_P0.5mm_EP3.5x3.5mm"
 			(at 168.91 120.65 0)
 			(effects
@@
 		(in_bom yes)
 		(on_board yes)
-		(dnp yes)
+		(dnp no)
 		(property "Reference" "C517"
 			(at 251.46 138.43 0)
@@
 		(in_bom yes)
 		(on_board yes)
-		(dnp yes)
+		(dnp no)
 		(fields_autoplaced yes)
 		(property "Reference" "C526"
@@
 		(in_bom yes)
 		(on_board yes)
-		(dnp yes)
+		(dnp no)
 		(fields_autoplaced yes)
 		(property "Reference" "R501"
@@
 		(in_bom yes)
 		(on_board yes)
-		(dnp yes)
+		(dnp no)
 		(property "Reference" "U505"
 			(at 142.24 68.58 0)
@@
 		(in_bom yes)
 		(on_board yes)
-		(dnp yes)
+		(dnp no)
 		(property "Reference" "C510"
 			(at 146.05 138.43 0)
@@
 		(in_bom yes)
 		(on_board yes)
-		(dnp yes)
+		(dnp no)
 		(property "Reference" "C506"
 			(at 105.41 138.43 0)
@@
 		(in_bom yes)
 		(on_board yes)
-		(dnp yes)
+		(dnp no)
 		(fields_autoplaced yes)
 		(property "Reference" "C523"
@@
 		(in_bom yes)
 		(on_board yes)
-		(dnp yes)
+		(dnp no)
 		(property "Reference" "C534"
 			(at 95.25 106.426 90)
@@
 		(in_bom yes)
 		(on_board yes)
-		(dnp yes)
+		(dnp no)
 		(fields_autoplaced yes)
 		(property "Reference" "C520"
@@
 		(in_bom yes)
 		(on_board yes)
-		(dnp yes)
+		(dnp no)
 		(fields_autoplaced yes)
 		(property "Reference" "R504"
@@
 		(in_bom yes)
 		(on_board yes)
-		(dnp yes)
+		(dnp no)
 		(property "Reference" "C512"
 			(at 200.66 138.43 0)
@@
 		(in_bom yes)
 		(on_board yes)
-		(dnp yes)
+		(dnp no)
 		(fields_autoplaced yes)
 		(property "Reference" "U503"
@@
 		(in_bom yes)
 		(on_board yes)
-		(dnp yes)
+		(dnp no)
 		(property "Reference" "C519"
 			(at 271.78 138.43 0)
@@
 		(in_bom yes)
 		(on_board yes)
-		(dnp yes)
+		(dnp no)
 		(property "Reference" "C508"
 			(at 125.73 138.43 0)
@@
 		(in_bom yes)
 		(on_board yes)
-		(dnp yes)
+		(dnp no)
 		(property "Reference" "U504"
 			(at 180.34 26.67 0)
@@
 		(in_bom yes)
 		(on_board yes)
-		(dnp yes)
+		(dnp no)
 		(fields_autoplaced yes)
 		(property "Reference" "C533"

Commit message: finaly working variants
Parts:
- A101: Var (none) -> Assembly Full(-!) Partial(+!); now fitted
- C501, C502, C503, C504, C505, C506, C507, C508, C509, C510, C511, C512, C513, C514, C515, C516, C517, C518, C519, C520, C521, C522, C523, C524, C525, C526, C527, C528, C531, C532, C533, C534, D502, J501, L501, L502, Q501, R501, R502, R503, R504, R505, U501, U502, U503, U505, Y501: Var (none) -> Assembly Full(+!) Partial(-!); now not fitted; now left out of the parts list
- U504, U506: Var (none) -> Assembly Full(-!) Partial(-!); now not fitted; now left out of the parts list

Commit message: cleanup
Parts:
- A101: now not fitted; now left out of the parts list
- C501, C502, C503, C504, C505, C506, C507, C508, C509, C510, C511, C512, C513, C514, C515, C516, C517, C518, C519, C520, C521, C522, C523, C524, C525, C526, C527, C528, C531, C532, C533, C534, D502, J501, L501, L502, Q501, R501, R502, R503, R504, R505, U502, U503, U505, Y501: now fitted; now in the parts list
- U501: symbol myParts:ST25R3916B -> additial parts:ST25R3916B; now fitted; now in the parts list
