File: Hardware/PCB/analog.kicad_sch (KiCad schematic)
At the start: 42 parts, among them J601 Conn_02x02_Odd_Even, J602 AudioJack3_SwitchTR, J603 Phoenix 1844236, J604 Conn_01x03, J605 AudioJack3_SwitchTR, SW601 CTS 218-4LPSTR, U601 TLV320AIC3104, U602 MAX98306xDT

Commit message: ~ hw-files update
Parts:
- C606, C622: Manufacturer (none) -> Kemet; Part Number (none) -> C0603C105K4RACTU
- C610, C611: Part Number (none) -> CL21A107MQYNNWE
- C614, C615, C620, R608, R609: now not fitted
- J602, J605: Part Number (none) -> SJ2-3593D-SMT-TR
Changed lines of the file:
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@@
 			)
 		)
+		(property "Part Number" "CL21A107MQYNNWE"
+			(at 142.24 29.21 90)
+			(effects
+				(font
+					(size 1.27 1.27)
+				)
+				(hide yes)
+			)
+		)
 		(pin "2"
 		)
@@
 		(in_bom yes)
 		(on_board yes)
-		(dnp no)
+		(dnp yes)
 		(property "Reference" "R608"
 			(at 217.17 144.78 0)
@@
 		(in_bom yes)
 		(on_board yes)
-		(dnp no)
+		(dnp yes)
 		(property "Reference" "R609"
 			(at 226.06 144.78 0)
@@
 			)
 		)
+		(property "Manufacturer" "Kemet"
+			(at 101.6 133.35 0)
+			(effects
+				(font
+					(size 1.27 1.27)
+				)
+				(hide yes)
+			)
+		)
+		(property "Part Number" "C0603C105K4RACTU"
+			(at 101.6 133.35 0)
+			(effects
+				(font
+					(size 1.27 1.27)
+				)
+				(hide yes)
+			)
+		)
 		(pin "2"
 		)
@@
 		(in_bom yes)
 		(on_board yes)
-		(dnp no)
+		(dnp yes)
 		(property "Reference" "C620"
 			(at 180.848 144.78 0)
@@
 			)
 		)
+		(property "Manufacturer" "Kemet"
+			(at 231.14 50.8 0)
+			(effects
+				(font
+					(size 1.27 1.27)
+				)
+				(hide yes)
+			)
+		)
+		(property "Part Number" "C0603C105K4RACTU"
+			(at 231.14 50.8 0)
+			(effects
+				(font
+					(size 1.27 1.27)
+				)
+				(hide yes)
+			)
+		)
 		(pin "2"
 		)
@@
 			)
 		)
+		(property "Part Number" "CL21A107MQYNNWE"
+			(at 142.24 24.13 90)
+			(effects
+				(font
+					(size 1.27 1.27)
+				)
+				(hide yes)
+			)
+		)
 		(pin "2"
 		)
@@
 			)
 		)
+		(property "Part Number" "SJ2-3593D-SMT-TR"
+			(at 242.57 133.35 0)
+			(effects
+				(font
+					(size 1.27 1.27)
+				)
+				(hide yes)
+			)
+		)
 		(pin "TN"
 		)
@@
 		(in_bom yes)
 		(on_board yes)
-		(dnp no)
+		(dnp yes)
 		(property "Reference" "C614"
 			(at 203.454 144.78 0)
@@
 		(in_bom yes)
 		(on_board yes)
-		(dnp no)
+		(dnp yes)
 		(property "Reference" "C615"
 			(at 192.024 144.78 0)
@@
 			(at 173.99 43.18 0)
 			(effects
+				(font
+					(size 1.27 1.27)
+				)
+				(hide yes)
+			)
+		)
+		(property "Part Number" "SJ2-3593D-SMT-TR"
+			(at 173.99 43.18 0)
+			(effects

Commit message: ~fixes on schematic and pcb ~prep for final output generation
Parts:
- added R612: 2k7, Resistor_SMD:R_0603_1608Metric_Pad0.98x0.95mm_HandSolder, symbol Device:R
- C601, C603, C605, C608, C612, C613, C621: Manufacturer (none) -> Kemet; Part Number (none) -> C0603C104K5RACTUCT
- C602, C604, C607, C609: Manufacturer (none) -> Kemet; Part Number (none) -> C0603C106M9PAC7411
- C610, C611: Manufacturer (none) -> Samsung Electro-Mechanics
- C614, C615, C620, R608, R609: Manufacturer (none) -> -; Part Number (none) -> -
- C616, C617, C618, C619: Manufacturer (none) -> Kemet; Part Number (none) -> C0603C473K5RACTUCT
- J601: Manufacturer (none) -> Würth Elektronik; Part Number (none) -> 61300421121
- J602, J605: Manufacturer (none) -> Same Sky (Formerly CUI Devices)
- J603: Manufacturer (none) -> Amphenol Anytek; Part Number (none) -> OQ041G01B000G, TJ0411030000G
- MK601: Manufacturer (none) -> Same Sky (Formerly CUI Devices); Part Number (none) -> CMA-4544PF-W
- R601, R602: Manufacturer (none) -> Yageo; Part Number (none) -> RC0603FR-072K2L
- R603: Manufacturer (none) -> Yageo; Part Number (none) -> RC0603FR-07100KL
- R604, R605, R606, R607: Manufacturer (none) -> Yageo; Part Number (none) -> RC0603FR-07100RL
- R610, R611: Manufacturer (none) -> Bourns Inc.; Part Number (none) -> CR0603AJ/-000EAS
- U601: Manufacturer (none) -> Texas Instruments; Part Number (none) -> TLV320AIC3104IRHBR
- U602: Manufacturer (none) -> Analog Devices Inc./Maxim Integrated; Part Number (none) -> MAX98306ETD+T
Connections:
- net +3V3: now also R612.1
- net at J601.2 (Pin_2), J601.4 (Pin_4), MK601.2 (+): now also R612.2
Other:
- moved on the sheet: MK601

Commit message: ~ board 3D files improved ~ bom output prep
Parts:
- J602, J605: footprint Connector_Audio:Jack_3.5mm_CUI_SJ2-3593D-SMT_Horizontal -> additional parts:Jack_3.5mm_CUI_SJ2-3593D-SMT_Horizontal
- J604: Manufacturer (none) -> Würth Elektronik; Part Number (none) -> 61300311121
- MK601: footprint Connector_PinHeader_2.54mm:PinHeader_1x02_P2.54mm_Vertical -> additional parts:Mic, dia 10mm pitch 2.54mm
- SW601: value CTS 218-4LPSTR -> CTS 218-4LPSTJ; footprint Package_SO:SSOP-8_3.9x5.05mm_P1.27mm -> additional parts:SSOP-8_3.9x5.05mm_P1.27mm; Manufacturer (none) -> CTS Electrocomponents; Part Number (none) -> 218-4LPSTJ
- U601: footprint Package_DFN_QFN:VQFN-32-1EP_5x5mm_P0.5mm_EP3.1x3.1mm -> additional parts:VQFN-32-1EP_5x5mm_P0.5mm_EP3.1x3.1mm
- U602: footprint Package_DFN_QFN:TDFN-14-1EP_3x3mm_P0.4mm_EP1.78x2.35mm -> additional parts:TDFN-14-1EP_3x3mm_P0.4mm_EP1.78x2.35mm
Changed lines of the file:
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@@
 			)
 		)
-		(property "Footprint" "Package_DFN_QFN:TDFN-14-1EP_3x3mm_P0.4mm_EP1.78x2.35mm"
+		(property "Footprint" "additional parts:TDFN-14-1EP_3x3mm_P0.4mm_EP1.78x2.35mm"
 			(at 209.55 69.85 0)
 			(effects
@@
 			)
 		)
-		(property "Value" "CTS 218-4LPSTR"
+		(property "Value" "CTS 218-4LPSTJ"
 			(at 142.24 35.56 0)
 			(effects
@@
 			)
 		)
-		(property "Footprint" "Package_SO:SSOP-8_3.9x5.05mm_P1.27mm"
+		(property "Footprint" "additional parts:SSOP-8_3.9x5.05mm_P1.27mm"
 			(at 142.24 45.72 0)
 			(effects
@@
 			)
 		)
+		(property "Manufacturer" "CTS Electrocomponents"
+			(at 142.24 45.72 0)
+			(effects
+				(font
+					(size 1.27 1.27)
+				)
+				(hide yes)
+			)
+		)
+		(property "Part Number" "218-4LPSTJ"
+			(at 142.24 45.72 0)
+			(effects
+				(font
+					(size 1.27 1.27)
+				)
+				(hide yes)
+			)
+		)
 		(pin "4"
 		)
@@
 			)
 		)
-		(property "Footprint" "Package_DFN_QFN:VQFN-32-1EP_5x5mm_P0.5mm_EP3.1x3.1mm"
+		(property "Footprint" "additional parts:VQFN-32-1EP_5x5mm_P0.5mm_EP3.1x3.1mm"
 			(at 103.124 31.496 0)
 			(effects
@@
 			)
 		)
-		(property "Footprint" "Connector_PinHeader_2.54mm:PinHeader_1x02_P2.54mm_Vertical"
+		(property "Footprint" "additional parts:Mic, dia 10mm pitch 2.54mm"
 			(at 269.24 109.22 90)
 			(effects
@@
 			)
 		)
-		(property "Footprint" "Package_DFN_QFN:VQFN-32-1EP_5x5mm_P0.5mm_EP3.1x3.1mm"
+		(property "Footprint" "additional parts:VQFN-32-1EP_5x5mm_P0.5mm_EP3.1x3.1mm"
 			(at 26.416 103.886 0)
 			(effects
@@
 			)
 		)
-		(property "Footprint" "Package_DFN_QFN:VQFN-32-1EP_5x5mm_P0.5mm_EP3.1x3.1mm"
+		(property "Footprint" "additional parts:VQFN-32-1EP_5x5mm_P0.5mm_EP3.1x3.1mm"
 			(at 55.626 31.496 0)
 			(effects
@@
 			)
 		)
-		(property "Footprint" "Package_DFN_QFN:VQFN-32-1EP_5x5mm_P0.5mm_EP3.1x3.1mm"
+		(property "Footprint" "additional parts:VQFN-32-1EP_5x5mm_P0.5mm_EP3.1x3.1mm"
 			(at 166.624 103.886 0)
 			(effects
@@
 			)
 		)
-		(property "Footprint" "Connector_Audio:Jack_3.5mm_CUI_SJ2-3593D-SMT_Horizontal"
+		(property "Footprint" "additional parts:Jack_3.5mm_CUI_SJ2-3593D-SMT_Horizontal"
 			(at 242.57 133.35 0)
 			(effects
@@
 			)
 		)
+		(property "Manufacturer" "Würth Elektronik"
+			(at 213.36 106.68 90)
+			(effects
+				(font
+					(size 1.27 1.27)
+				)
+				(hide yes)
+			)
+		)
+		(property "Part Number" "61300311121"
+			(at 213.36 106.68 90)
+			(effects
+				(font
+					(size 1.27 1.27)
+				)
+				(hide yes)
+			)
+		)
 		(pin "2"
 		)
@@
 			)
 		)
-		(property "Footprint" "Connector_Audio:Jack_3.5mm_CUI_SJ2-3593D-SMT_Horizontal"
+		(property "Footprint" "additional parts:Jack_3.5mm_CUI_SJ2-3593D-SMT_Horizontal"
 			(at 173.99 43.18 0)
 			(effects

Commit message: cleanup
Parts:
- U601: footprint additional parts:VQFN-32-1EP_5x5mm_P0.5mm_EP3.1x3.1mm -> Package_DFN_QFN:VQFN-32-1EP_5x5mm_P0.5mm_EP3.1x3.1mm; symbol myParts:TLV320AIC3104 -> additial parts:TLV320AIC3104
Changed lines of the file:
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@@
 	)
 	(symbol
-		(lib_id "myParts:TLV320AIC3104")
+		(lib_id "additial parts:TLV320AIC3104")
 		(at 107.95 39.37 0)
 		(mirror y)
@@
 			)
 		)
-		(property "Footprint" "additional parts:VQFN-32-1EP_5x5mm_P0.5mm_EP3.1x3.1mm"
+		(property "Footprint" "Package_DFN_QFN:VQFN-32-1EP_5x5mm_P0.5mm_EP3.1x3.1mm"
 			(at 103.124 31.496 0)
 			(effects
@@
 	)
 	(symbol
-		(lib_id "myParts:TLV320AIC3104")
+		(lib_id "additial parts:TLV320AIC3104")
 		(at 21.59 111.76 0)
 		(unit 4)
@@
 			)
 		)
-		(property "Footprint" "additional parts:VQFN-32-1EP_5x5mm_P0.5mm_EP3.1x3.1mm"
+		(property "Footprint" "Package_DFN_QFN:VQFN-32-1EP_5x5mm_P0.5mm_EP3.1x3.1mm"
 			(at 26.416 103.886 0)
 			(effects
@@
 	)
 	(symbol
-		(lib_id "myParts:TLV320AIC3104")
+		(lib_id "additial parts:TLV320AIC3104")
 		(at 50.8 39.37 0)
 		(unit 3)
@@
 			)
 		)
-		(property "Footprint" "additional parts:VQFN-32-1EP_5x5mm_P0.5mm_EP3.1x3.1mm"
+		(property "Footprint" "Package_DFN_QFN:VQFN-32-1EP_5x5mm_P0.5mm_EP3.1x3.1mm"
 			(at 55.626 31.496 0)
 			(effects
@@
 	)
 	(symbol
-		(lib_id "myParts:TLV320AIC3104")
+		(lib_id "additial parts:TLV320AIC3104")
 		(at 171.45 111.76 0)
 		(mirror y)
@@
 			)
 		)
-		(property "Footprint" "additional parts:VQFN-32-1EP_5x5mm_P0.5mm_EP3.1x3.1mm"
+		(property "Footprint" "Package_DFN_QFN:VQFN-32-1EP_5x5mm_P0.5mm_EP3.1x3.1mm"
 			(at 166.624 103.886 0)
 			(effects
