File: Hardware/PCB/pinout.kicad_sch (KiCad schematic)
At the start: 5 parts, among them CN201 Conn_02x08_Odd_Even

Commit message: ~fixes on schematic and pcb ~prep for final output generation
Parts:
- CN202: footprint Connector_PinSocket_2.54mm:PinSocket_2x08_P2.54mm_Vertical -> Connector_PinHeader_2.54mm:PinHeader_2x08_P2.54mm_Vertical; Manufacturer (none) -> Würth Elektronik; Part Number (none) -> 61301621121
- CN203: footprint Connector_PinSocket_2.54mm:PinSocket_2x15_P2.54mm_Vertical -> Connector_PinHeader_2.54mm:PinHeader_2x15_P2.54mm_Vertical; Manufacturer (none) -> Samtec Inc.; Part Number (none) -> TSW-115-24-L-D
- CN204: footprint Connector_PinSocket_2.54mm:PinSocket_2x10_P2.54mm_Vertical -> Connector_PinHeader_2.54mm:PinHeader_2x10_P2.54mm_Vertical; Manufacturer (none) -> Adam Tech; Part Number (none) -> PH2-20-UA
- CN205: footprint Connector_PinSocket_2.54mm:PinSocket_2x17_P2.54mm_Vertical -> Connector_PinHeader_2.54mm:PinHeader_2x17_P2.54mm_Vertical; Manufacturer (none) -> Amphenol ICC (FCI); Part Number (none) -> 67997-234HLF
Connections:
- net +3V3: now also CN202.4 (IOREF), CN202.8 (+3V3); no longer CN202.3 (IOREF), CN202.7 (+3V3)
- net +5V: now also CN202.10 (+5V); no longer CN202.9 (+5V)
- net AREF: now also CN204.5 (VREFP); no longer CN204.6 (VREFP)
- net BTN0: now also CN204.17 (D9); no longer CN204.18 (D9)
- net BTN1: now also CN205.5 (D5); no longer CN205.6 (D5)
- net BTN2: now also CN205.7 (D4); no longer CN205.8 (D4)
- net BTN3: now also CN205.9 (D3); no longer CN205.10 (D3)
- net CODEC_nRESET: now also CN205.11 (D2); no longer CN205.12 (D2)
- net GND: now also CN202.12 (GND), CN202.14 (GND), CN203.11 (GND), CN203.24 (GND), CN204.7 (GND), CN205.18 (GND), CN205.21 (GND), CN205.28 (GND), CN205.4 (AGND), CN205.6 (GND); no longer CN202.11 (GND), CN202.13 (GND), CN203.12 (GND), CN203.23 (GND), CN204.8 (GND), CN205.17 (GND), CN205.22 (GND), CN205.27 (GND), CN205.3 (AGND), CN205.5 (GND)
- net I2C_SCL: now also CN204.1 (D15); no longer CN204.2 (D15)
- net I2C_SDA: now also CN204.3 (D14); no longer CN204.4 (D14)
- net I2S2_SDA_ext: now also CN203.4 (A1); no longer CN203.3 (A1)
- net I2S_BCLK: now also CN204.6 (D18); no longer CN204.5 (D18)
- net I2S_MCLK: now also CN204.2 (D16); no longer CN204.1 (D16)
- net I2S_SDA: now also CN204.4 (D17); no longer CN204.3 (D17)
- net I2S_SDA_ext: now also CN203.30 (D65); no longer CN204.19 (D25)
- net I2S_WCLK: now also CN204.8 (D19); no longer CN204.7 (D19)
- net INT: now also CN203.10 (A4); no longer CN203.9 (A4)
- net LED0: now also CN205.3 (D6); no longer CN205.4 (D6)
- net LED1: now also CN205.1 (D7); no longer CN205.2 (D7)
- net MISO: now also CN204.11 (D12); no longer CN204.12 (D12)
- net MOSI: now also CN204.13 (D11); no longer CN204.14 (D11)
- net NFC_INT: now also CN203.2 (A0); no longer CN203.1 (A0)
- net NSS: now also CN204.15 (D10); no longer CN204.16 (D10)
- net POT0: now also CN203.8 (A3); no longer CN203.7 (A3)
- net POT1: now also CN203.6 (A2); no longer CN203.5 (A2)
- net RX: now also CN205.15 (D0); no longer CN205.16 (D0)
- net SCK: now also CN204.9 (D13); no longer CN204.10 (D13)
- net SD_CLK: now also CN202.9 (D47); no longer CN202.10 (D47)
- net SD_CMD: now also CN202.11 (D48); no longer CN202.12 (D48)
- net SD_DAT0: now also CN202.1 (D43); no longer CN202.2 (D43)
- net SD_DAT1: now also CN202.3 (D44); no longer CN202.4 (D44)
- net SD_DAT2: now also CN202.5 (D45); no longer CN202.6 (D45)
- net SD_DAT3: now also CN202.7 (D46); no longer CN202.8 (D46)
- net SD_DET: now also CN202.13 (D49); no longer CN202.14 (D49)
- net SPI2_MISO: now also CN204.19 (D8); no longer CN204.20 (D8)
- net SPI2_MOSI: now also CN204.14 (D22); no longer CN204.13 (D22)
- net SPI2_NSS: now also CN204.18 (D24); no longer CN204.17 (D24)
- net SPI2_SCK: now also CN204.16 (D23); no longer CN204.15 (D23)
- net TX: now also CN205.13 (D1); no longer CN205.14 (D1)
- net ~{RESET}: now also CN202.6 (NRST); no longer CN202.5 (NRST)
Other:
- note added: "PB14"
Changed lines of the file:
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@@
 		)
 	)
-	(text "PB4"
-		(exclude_from_sim no)
-		(at 197.866 52.07 0)
-		(effects
-			(font
-				(face "Courier 10 Pitch")
-				(size 1.27 1.27)
-			)
-			(justify left bottom)
-		)
-	)
 	(text "PC1"
 		(exclude_from_sim no)
@@
 		)
 	)
+	(text "PB14"
+		(exclude_from_sim no)
+		(at 44.45 101.6 0)
+		(effects
+			(font
+				(face "Courier 10 Pitch")
+				(size 1.27 1.27)
+			)
+			(justify left bottom)
+		)
+	)
 	(text "PB7  | PG9"
 		(exclude_from_sim no)
@@
 	)
 	(no_connect
-		(at 66.04 101.6)
-	)
-	(no_connect
 		(at 209.55 92.71)
 	)
@@
 		(at 66.04 48.26)
 	)
+	(no_connect
+		(at 209.55 52.07)
+	)
 	(bus_entry
 		(at 143.51 35.56)
@@
 	(wire
 		(pts
+			(xy 30.48 101.6) (xy 66.04 101.6)
+		)
+		(stroke
+			(width 0)
+			(type default)
+		)
+	)
+	(wire
+		(pts
 			(xy 58.42 25.4) (xy 58.42 40.64)
 		)
@@
 	(wire
 		(pts
-			(xy 193.04 52.07) (xy 209.55 52.07)
-		)
-		(stroke
-			(width 0)
-			(type default)
-		)
-	)
-	(wire
-		(pts
 			(xy 86.36 43.18) (xy 116.84 43.18)
 		)
@@
 		)
 	)
+	(hierarchical_label "I2S_SDA_ext"
+		(shape bidirectional)
+		(at 30.48 101.6 180)
+		(effects
+			(font
+				(size 1.27 1.27)
+			)
+			(justify right)
+		)
+	)
 	(hierarchical_label "I2S_MCLK"
 		(shape bidirectional)
@@
 		)
 	)
-	(hierarchical_label "I2S_SDA_ext"
-		(shape bidirectional)
-		(at 193.04 52.07 180)
-		(effects
-			(font
-				(size 1.27 1.27)
-			)
-			(justify right)
-		)
-	)
 	(hierarchical_label "CODEC_nRESET"
 		(shape bidirectional)
@@
 			)
 		)
-		(property "Footprint" "Connector_PinSocket_2.54mm:PinSocket_2x08_P2.54mm_Vertical"
+		(property "Footprint" "Connector_PinHeader_2.54mm:PinHeader_2x08_P2.54mm_Vertical"
 			(at 68.58 29.21 0)
 			(effects
@@
 			)
 		)
+		(property "Manufacturer" "Würth Elektronik"
+			(at 68.58 29.21 0)
+			(effects
+				(font
+					(size 1.27 1.27)
+				)
+				(hide yes)
+			)
+		)
+		(property "Part Number" "61301621121"
+			(at 68.58 29.21 0)
+			(effects
+				(font
+					(size 1.27 1.27)
+				)
+				(hide yes)
+			)
+		)
 		(pin "8"
 		)
@@
 			)
 		)
-		(property "Footprint" "Connector_PinSocket_2.54mm:PinSocket_2x15_P2.54mm_Vertical"
+		(property "Footprint" "Connector_PinHeader_2.54mm:PinHeader_2x15_P2.54mm_Vertical"
 			(at 68.58 64.77 0)
 			(effects
@@
 			)
 		)
+		(property "Manufacturer" "Samtec Inc."
+			(at 68.58 64.77 0)
+			(effects
+				(font
+					(size 1.27 1.27)
+				)
+				(hide yes)
+			)
+		)
+		(property "Part Number" "TSW-115-24-L-D"
+			(at 68.58 64.77 0)
+			(effects
+				(font
+					(size 1.27 1.27)
+				)
+				(hide yes)
+			)
+		)
 		(pin "8"
 		)
@@
 			)
 		)
-		(property "Footprint" "Connector_PinSocket_2.54mm:PinSocket_2x17_P2.54mm_Vertical"
+		(property "Footprint" "Connector_PinHeader_2.54mm:PinHeader_2x17_P2.54mm_Vertical"
 			(at 212.09 63.5 0)
 			(effects
@@
 			)
 		)
+		(property "Manufacturer" "Amphenol ICC (FCI)"
+			(at 212.09 63.5 0)
+			(effects
+				(font
+					(size 1.27 1.27)
+				)
+				(hide yes)
+			)
+		)
+		(property "Part Number" "67997-234HLF"
+			(at 212.09 63.5 0)
+			(effects
+				(font
+					(size 1.27 1.27)
+				)
+				(hide yes)
+			)
+		)
 		(pin "20"
 		)
@@
 			)
 		)
-		(property "Footprint" "Connector_PinSocket_2.54mm:PinSocket_2x10_P2.54mm_Vertical"
+		(property "Footprint" "Connector_PinHeader_2.54mm:PinHeader_2x10_P2.54mm_Vertical"
 			(at 212.09 27.94 0)
 			(effects
@@
 			(at 212.09 27.94 0)
 			(effects
+				(font
+					(size 1.27 1.27)
+				)
+				(hide yes)
+			)
+		)
+		(property "Manufacturer" "Adam Tech"
+			(at 212.09 27.94 0)
+			(effects
+				(font
+					(size 1.27 1.27)
+				)
+				(hide yes)
+			)
+		)
+		(property "Part Number" "PH2-20-UA"
+			(at 212.09 27.94 0)
+			(effects

Commit message: ~ board 3D files improved ~ bom output prep
Parts:
- CN201: Manufacturer (none) -> Würth Elektronik; Part Number (none) -> 61301621821
Changed lines of the file:
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@@
+			)
+		)
+		(property "Manufacturer" "Würth Elektronik"
+			(at 49.53 144.78 0)
+			(effects
+				(font
+					(size 1.27 1.27)
+				)
+				(hide yes)
+			)
+		)
+		(property "Part Number" "61301621821"
+			(at 49.53 144.78 0)
+			(effects
+				(font
+					(size 1.27 1.27)
+				)
+				(hide yes)
 			)
 		)

Commit message: cleanup
Parts:
- CN202: symbol myParts:NUCLEO_144_Power -> additial parts:NUCLEO_144_Power
- CN203: symbol myParts:NUCLEO_144_Analog+ -> additial parts:NUCLEO_144_Analog+
- CN204: symbol myParts:NUCLEO_144_Periphery+ -> additial parts:NUCLEO_144_Periphery+
- CN205: symbol myParts:NUCLEO_144_GPIO+ -> additial parts:NUCLEO_144_GPIO+
Changed lines of the file:
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@@
 	)
 	(symbol
-		(lib_id "myParts:NUCLEO_144_Power")
+		(lib_id "additial parts:NUCLEO_144_Power")
 		(at 68.58 29.21 0)
 		(unit 1)
@@
 	)
 	(symbol
-		(lib_id "myParts:NUCLEO_144_Analog+")
+		(lib_id "additial parts:NUCLEO_144_Analog+")
 		(at 68.58 64.77 0)
 		(unit 1)
@@
 	)
 	(symbol
-		(lib_id "myParts:NUCLEO_144_GPIO+")
+		(lib_id "additial parts:NUCLEO_144_GPIO+")
 		(at 212.09 63.5 0)
 		(unit 1)
@@
 	)
 	(symbol
-		(lib_id "myParts:NUCLEO_144_Periphery+")
+		(lib_id "additial parts:NUCLEO_144_Periphery+")
 		(at 212.09 27.94 0)
 		(unit 1)
