File: Hardware/PCB/wireless.kicad_sch (KiCad schematic)
At the start: 9 parts, among them J301 Conn_02x06_Top_Bottom, J302 Conn_02x06_Odd_Even, J303 Conn_01x06, U301 ESP32-WROOM-32

Commit message: ~ hw-files update
Parts:
- removed J301: Conn_02x06_Top_Bottom, Connector_PinHeader_2.54mm:PinHeader_2x06_P2.54mm_Horizontal, symbol Connector_Generic:Conn_02x06_Top_Bottom
- J301: renamed from J302; footprint (none) -> Connector_PinHeader_2.54mm:PinHeader_2x06_P2.54mm_Horizontal
Connections:
- net +3V3: now also J301.11 (Pin_11), J301.12 (Pin_12)
- net EN: now also J301.4 (Pin_4)
- net GND: now also J301.10 (Pin_10), J301.9 (Pin_9); no longer R303.2
- net GPIO: now also J301.8 (Pin_8)
- net INT: now also J301.2 (Pin_2)
- net IO0: no longer J303.2 (Pin_2)
- net MISO: now also J301.5 (Pin_5)
- net MOSI: now also J301.3 (Pin_3)
- net NSS: now also J301.1 (Pin_1)
- net SCK: now also J301.7 (Pin_7)
- net SELECT: now also J301.6 (Pin_6)
- new net: J303.2 (Pin_2), R303.2
Other:
- note added: "set to Boot mode connect Pin2 & Pin3"
- note removed: "Compare"
- note removed: "set Boot-mode (2) to high"
- moved on the sheet: J301, R303
Changed lines of the file:
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@@
 	(generator_version "9.0")
 	(paper "A4")
-	(text "set Boot-mode (2) to high"
+	(text "set to Boot mode\nconnect Pin2 & Pin3"
 		(exclude_from_sim no)
-		(at 235.204 61.214 0)
+		(at 235.204 59.69 0)
 		(effects
 			(font
@@
 		(exclude_from_sim no)
 		(at 230.886 55.118 0)
-		(effects
-			(font
-				(size 1.27 1.27)
-			)
-			(justify left)
-		)
-	)
-	(text "Compare"
-		(exclude_from_sim no)
-		(at 120.396 26.162 0)
 		(effects
 			(font
@@
 	)
 	(junction
-		(at 203.2 71.12)
-		(diameter 0)
-		(color 0 0 0 0)
-	)
-	(junction
 		(at 185.42 60.96)
 		(diameter 0)
@@
 	)
 	(junction
-		(at 203.2 60.96)
-		(diameter 0)
-		(color 0 0 0 0)
-	)
-	(junction
 		(at 137.16 41.91)
 		(diameter 0)
@@
 	(wire
 		(pts
-			(xy 203.2 69.85) (xy 203.2 71.12)
-		)
-		(stroke
-			(width 0)
-			(type default)
-		)
-	)
-	(wire
-		(pts
 			(xy 119.38 83.82) (xy 119.38 68.58)
 		)
@@
 	(wire
 		(pts
-			(xy 227.33 63.5) (xy 210.82 63.5)
+			(xy 203.2 63.5) (xy 203.2 72.39)
 		)
 		(stroke
@@
 	(wire
 		(pts
-			(xy 210.82 63.5) (xy 210.82 71.12)
-		)
-		(stroke
-			(width 0)
-			(type default)
-		)
-	)
-	(wire
-		(pts
 			(xy 217.17 66.04) (xy 227.33 66.04)
 		)
@@
 	(wire
 		(pts
+			(xy 209.55 60.96) (xy 227.33 60.96)
+		)
+		(stroke
+			(width 0)
+			(type default)
+		)
+	)
+	(wire
+		(pts
 			(xy 137.16 41.91) (xy 137.16 48.26)
 		)
@@
 	(wire
 		(pts
-			(xy 203.2 71.12) (xy 203.2 72.39)
-		)
-		(stroke
-			(width 0)
-			(type default)
-		)
-	)
-	(wire
-		(pts
 			(xy 96.52 71.12) (xy 102.87 71.12)
 		)
@@
 	(wire
 		(pts
-			(xy 203.2 60.96) (xy 203.2 62.23)
-		)
-		(stroke
-			(width 0)
-			(type default)
-		)
-	)
-	(wire
-		(pts
 			(xy 227.33 71.12) (xy 224.79 71.12)
 		)
@@
 	(wire
 		(pts
+			(xy 227.33 63.5) (xy 203.2 63.5)
+		)
+		(stroke
+			(width 0)
+			(type default)
+		)
+	)
+	(wire
+		(pts
 			(xy 195.58 93.98) (xy 177.8 93.98)
 		)
@@
 	(wire
 		(pts
-			(xy 185.42 60.96) (xy 203.2 60.96)
+			(xy 185.42 60.96) (xy 201.93 60.96)
 		)
 		(stroke
@@
 	(wire
 		(pts
-			(xy 203.2 71.12) (xy 210.82 71.12)
-		)
-		(stroke
-			(width 0)
-			(type default)
-		)
-	)
-	(wire
-		(pts
 			(xy 195.58 106.68) (xy 177.8 106.68)
 		)
@@
 		(pts
 			(xy 54.61 63.5) (xy 78.74 63.5)
-		)
-		(stroke
-			(width 0)
-			(type default)
-		)
-	)
-	(wire
-		(pts
-			(xy 203.2 60.96) (xy 227.33 60.96)
 		)
 		(stroke
@@
 	)
 	(label "IO0"
-		(at 210.82 60.96 180)
+		(at 198.12 60.96 180)
 		(effects
 			(font
@@
 	(symbol
 		(lib_id "Device:R")
-		(at 203.2 66.04 0)
+		(at 205.74 60.96 90)
 		(unit 1)
 		(exclude_from_sim no)
@@
 		(fields_autoplaced yes)
 		(property "Reference" "R303"
-			(at 205.74 64.7699 0)
-			(effects
-				(font
-					(size 1.27 1.27)
-				)
-				(justify left)
+			(at 205.74 54.61 90)
+			(effects
+				(font
+					(size 1.27 1.27)
+				)
 			)
 		)
 		(property "Value" "1k"
-			(at 205.74 67.3099 0)
-			(effects
-				(font
-					(size 1.27 1.27)
-				)
-				(justify left)
+			(at 205.74 57.15 90)
+			(effects
+				(font
+					(size 1.27 1.27)
+				)
 			)
 		)
 		(property "Footprint" "Resistor_SMD:R_0805_2012Metric_Pad1.20x1.40mm_HandSolder"
-			(at 201.422 66.04 90)
+			(at 205.74 62.738 90)
 			(effects
 				(font
@@
 		)
 		(property "Datasheet" "~"
-			(at 203.2 66.04 0)
+			(at 205.74 60.96 0)
 			(effects
 				(font
@@
 		)
 		(property "Description" "Resistor"
-			(at 203.2 66.04 0)
+			(at 205.74 60.96 0)
 			(effects
 				(font
@@
 	(symbol
 		(lib_id "Connector_Generic:Conn_02x06_Odd_Even")
-		(at 107.95 26.67 0)
+		(at 107.95 63.5 0)
 		(unit 1)
 		(exclude_from_sim no)
@@
 		(dnp no)
 		(fields_autoplaced yes)
-		(property "Reference" "J302"
-			(at 109.22 15.24 0)
+		(property "Reference" "J301"
+			(at 109.22 52.07 0)
 			(effects
 				(font
@@
 		)
 		(property "Value" "Conn_02x06_Odd_Even"
-			(at 109.22 17.78 0)
-			(effects
-				(font
-					(size 1.27 1.27)
-				)
-			)
-		)
-		(property "Footprint" ""
-			(at 107.95 26.67 0)
+			(at 109.22 54.61 0)
+			(effects
+				(font
+					(size 1.27 1.27)
+				)
+			)
+		)
+		(property "Footprint" "Connector_PinHeader_2.54mm:PinHeader_2x06_P2.54mm_Horizontal"
+			(at 107.95 63.5 0)
 			(effects
 				(font
@@
 		)
 		(property "Datasheet" "~"
-			(at 107.95 26.67 0)
+			(at 107.95 63.5 0)
 			(effects
 				(font
@@
 		)
 		(property "Description" "Generic connector, double row, 02x06, odd/even pin numbering scheme (row 1 odd numbers, row 2 even numbers), script generated (kicad-library-utils/schlib/autogen/connector/)"
-			(at 107.95 26.67 0)
+			(at 107.95 63.5 0)
 			(effects
 				(font
@@
 			(project ""
 				(path "/e63e39d7-6ac0-4ffd-8aa3-1841a4541b55/c4907074-0e50-41f9-8f09-d9d4d6cc7ba3"
-					(reference "J302")
-					(unit 1)
-				)
-			)
-		)
-	)
-	(symbol
-		(lib_id "Connector_Generic:Conn_02x06_Top_Bottom")
-		(at 107.95 63.5 0)
-		(unit 1)
-		(exclude_from_sim no)
-		(in_bom yes)
-		(on_board yes)
-		(dnp no)
-		(property "Reference" "J301"
-			(at 109.22 52.07 0)
-			(effects
-				(font
-					(size 1.27 1.27)
-				)
-			)
-		)
-		(property "Value" "Conn_02x06_Top_Bottom"
-			(at 109.22 54.61 0)
-			(effects
-				(font
-					(size 1.27 1.27)
-				)
-			)
-		)
-		(property "Footprint" "Connector_PinHeader_2.54mm:PinHeader_2x06_P2.54mm_Horizontal"
-			(at 107.95 63.5 0)
-			(effects
-				(font
-					(size 1.27 1.27)
-				)
-				(hide yes)
-			)
-		)
-		(property "Datasheet" "~"
-			(at 107.95 63.5 0)
-			(effects
-				(font
-					(size 1.27 1.27)
-				)
-				(hide yes)
-			)
-		)
-		(property "Description" "Generic connector, double row, 02x06, top/bottom pin numbering scheme (row 1: 1...pins_per_row, row2: pins_per_row+1 ... num_pins), script generated (kicad-library-utils/schlib/autogen/connector/)"
-			(at 107.95 63.5 0)
-			(effects
-				(font
-					(size 1.27 1.27)
-				)
-				(hide yes)
-			)
-		)
-		(pin "7"
-		)
-		(pin "12"
-		)
-		(pin "1"
-		)
-		(pin "2"
-		)
-		(pin "10"
-		)
-		(pin "9"
-		)
-		(pin "8"
-		)
-		(pin "4"
-		)
-		(pin "6"
-		)
-		(pin "3"
-		)
-		(pin "5"
-		)
-		(pin "11"
-		)
-		(instances
-			(project "voicemail-box"
-				(path "/e63e39d7-6ac0-4ffd-8aa3-1841a4541b55/c4907074-0e50-41f9-8f09-d9d4d6cc7ba3"
 					(reference "J301")

Commit message: ~fixes on schematic and pcb ~prep for final output generation
Parts:
- C301: Manufacturer (none) -> Kemet; Part Number (none) -> C0805C104K5RACTU; now not fitted
- C302: Manufacturer (none) -> Kemet; Part Number (none) -> C0603C106M9PAC7411; now not fitted
- J303: now not fitted
- R301: Manufacturer (none) -> Yageo; Part Number (none) -> RC0603FR-0710KL; now not fitted
- R302: Manufacturer (none) -> Yageo; Part Number (none) -> RC0603FR-0720KL; now not fitted
- R303: Manufacturer (none) -> Yageo; Part Number (none) -> RC0603FR-071KL; now not fitted
- U301: Manufacturer (none) -> Espressif Systems; Part Number (none) -> ESP32-WROOM-32E-H4; now not fitted
Changed lines of the file:
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@@
 		(in_bom yes)
 		(on_board yes)
-		(dnp no)
+		(dnp yes)
 		(property "Reference" "C301"
 			(at 145.796 44.45 0)
@@
 			)
 		)
+		(property "Manufacturer" "Kemet"
+			(at 144.78 46.99 0)
+			(effects
+				(font
+					(size 1.27 1.27)
+				)
+				(hide yes)
+			)
+		)
+		(property "Part Number" "C0805C104K5RACTU"
+			(at 144.78 46.99 0)
+			(effects
+				(font
+					(size 1.27 1.27)
+				)
+				(hide yes)
+			)
+		)
 		(pin "1"
 		)
@@
 		(in_bom yes)
 		(on_board yes)
-		(dnp no)
+		(dnp yes)
 		(property "Reference" "C302"
 			(at 157.48 44.196 0)
@@
 		)
 		(property "Description" "Unpolarized capacitor"
+			(at 156.21 46.99 0)
+			(effects
+				(font
+					(size 1.27 1.27)
+				)
+				(hide yes)
+			)
+		)
+		(property "Manufacturer" "Kemet"
+			(at 156.21 46.99 0)
+			(effects
+				(font
+					(size 1.27 1.27)
+				)
+				(hide yes)
+			)
+		)
+		(property "Part Number" "C0603C106M9PAC7411"
 			(at 156.21 46.99 0)
 			(effects
@@
 		(in_bom yes)
 		(on_board yes)
-		(dnp no)
+		(dnp yes)
 		(fields_autoplaced yes)
 		(property "Reference" "R303"
@@
 		(property "Description" "Resistor"
 			(at 205.74 60.96 0)
+			(effects
+				(font
+					(size 1.27 1.27)
+				)
+				(hide yes)
+			)
+		)
+		(property "Manufacturer" "Yageo"
+			(at 205.74 60.96 90)
+			(effects
+				(font
+					(size 1.27 1.27)
+				)
+				(hide yes)
+			)
+		)
+		(property "Part Number" "RC0603FR-071KL"
+			(at 205.74 60.96 90)
 			(effects
 				(font
@@
 		(in_bom yes)
 		(on_board yes)
-		(dnp no)
+		(dnp yes)
 		(fields_autoplaced yes)
 		(property "Reference" "R302"
@@
 			)
 		)
+		(property "Manufacturer" "Yageo"
+			(at 185.42 52.07 0)
+			(effects
+				(font
+					(size 1.27 1.27)
+				)
+				(hide yes)
+			)
+		)
+		(property "Part Number" "RC0603FR-0720KL"
+			(at 185.42 52.07 0)
+			(effects
+				(font
+					(size 1.27 1.27)
+				)
+				(hide yes)
+			)
+		)
 		(pin "2"
 		)
@@
 		(in_bom yes)
 		(on_board yes)
-		(dnp no)
+		(dnp yes)
 		(fields_autoplaced yes)
 		(property "Reference" "R301"
@@
 		)
 		(property "Description" "Resistor"
+			(at 137.16 52.07 0)
+			(effects
+				(font
+					(size 1.27 1.27)
+				)
+				(hide yes)
+			)
+		)
+		(property "Manufacturer" "Yageo"
+			(at 137.16 52.07 0)
+			(effects
+				(font
+					(size 1.27 1.27)
+				)
+				(hide yes)
+			)
+		)
+		(property "Part Number" "RC0603FR-0710KL"
 			(at 137.16 52.07 0)
 			(effects
@@
 		(in_bom yes)
 		(on_board yes)
-		(dnp no)
+		(dnp yes)
 		(property "Reference" "U301"
 			(at 165.1 54.864 0)
@@
 		)
 		(property "Description" "RF Module, ESP32-D0WDQ6 SoC, Wi-Fi 802.11b/g/n, Bluetooth, BLE, 32-bit, 2.7-3.6V, onboard antenna, SMD"
+			(at 162.56 91.44 0)
+			(effects
+				(font
+					(size 1.27 1.27)
+				)
+				(hide yes)
+			)
+		)
+		(property "Manufacturer" "Espressif Systems"
+			(at 162.56 91.44 0)
+			(effects
+				(font
+					(size 1.27 1.27)
+				)
+				(hide yes)
+			)
+		)
+		(property "Part Number" "ESP32-WROOM-32E-H4"
 			(at 162.56 91.44 0)
 			(effects
@@
 		(in_bom yes)
 		(on_board yes)
-		(dnp no)
+		(dnp yes)
 		(fields_autoplaced yes)
 		(property "Reference" "J303"

Commit message: ~ board 3D files improved ~ bom output prep
Parts:
- C301, C302, R301, R302, R303, U301: now fitted
- J301: footprint Connector_PinHeader_2.54mm:PinHeader_2x06_P2.54mm_Horizontal -> additional parts:PinSocket_2x06_P2.54mm_Horizontal; Manufacturer (none) -> Würth Elektronik; Part Number (none) -> 613012243121; now not fitted
- J303: Manufacturer (none) -> Würth Elektronik; Part Number (none) -> 61300611121; now fitted
Changed lines of the file:
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@@
 		(in_bom yes)
 		(on_board yes)
-		(dnp yes)
+		(dnp no)
 		(property "Reference" "C301"
 			(at 145.796 44.45 0)
@@
 		(in_bom yes)
 		(on_board yes)
-		(dnp yes)
+		(dnp no)
 		(property "Reference" "C302"
 			(at 157.48 44.196 0)
@@
 		(in_bom yes)
 		(on_board yes)
-		(dnp yes)
+		(dnp no)
 		(fields_autoplaced yes)
 		(property "Reference" "R303"
@@
 		(in_bom yes)
 		(on_board yes)
-		(dnp yes)
+		(dnp no)
 		(fields_autoplaced yes)
 		(property "Reference" "R302"
@@
 		(in_bom yes)
 		(on_board yes)
-		(dnp yes)
+		(dnp no)
 		(fields_autoplaced yes)
 		(property "Reference" "R301"
@@
 		(in_bom yes)
 		(on_board yes)
-		(dnp yes)
+		(dnp no)
 		(property "Reference" "U301"
 			(at 165.1 54.864 0)
@@
 		(in_bom yes)
 		(on_board yes)
-		(dnp no)
+		(dnp yes)
 		(fields_autoplaced yes)
 		(property "Reference" "J301"
@@
 			)
 		)
-		(property "Footprint" "Connector_PinHeader_2.54mm:PinHeader_2x06_P2.54mm_Horizontal"
+		(property "Footprint" "additional parts:PinSocket_2x06_P2.54mm_Horizontal"
 			(at 107.95 63.5 0)
 			(effects
@@
 		)
 		(property "Description" "Generic connector, double row, 02x06, odd/even pin numbering scheme (row 1 odd numbers, row 2 even numbers), script generated (kicad-library-utils/schlib/autogen/connector/)"
+			(at 107.95 63.5 0)
+			(effects
+				(font
+					(size 1.27 1.27)
+				)
+				(hide yes)
+			)
+		)
+		(property "Manufacturer" "Würth Elektronik"
+			(at 107.95 63.5 0)
+			(effects
+				(font
+					(size 1.27 1.27)
+				)
+				(hide yes)
+			)
+		)
+		(property "Part Number" "613012243121"
 			(at 107.95 63.5 0)
 			(effects
@@
 		(in_bom yes)
 		(on_board yes)
-		(dnp yes)
+		(dnp no)
 		(fields_autoplaced yes)
 		(property "Reference" "J303"
@@
 			(at 232.41 63.5 0)
 			(effects
+				(font
+					(size 1.27 1.27)
+				)
+				(hide yes)
+			)
+		)
+		(property "Manufacturer" "Würth Elektronik"
+			(at 232.41 63.5 0)
+			(effects
+				(font
+					(size 1.27 1.27)
+				)
+				(hide yes)
+			)
+		)
+		(property "Part Number" "61300611121"
+			(at 232.41 63.5 0)
+			(effects

Commit message: finaly working variants
Parts:
- C301, J303, R301, R302, R303, U301: Var (none) -> Assembly Full(+!) Partial(-!); now not fitted; now left out of the parts list
- C302: Var (none) -> Assembly Full(-!) Partial(+!)
- J301: Var (none) -> Assembly Full(-!) Partial(+!); now fitted
Changed lines of the file:
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@@
 		(unit 1)
 		(exclude_from_sim no)
-		(in_bom yes)
-		(on_board yes)
-		(dnp no)
+		(in_bom no)
+		(on_board yes)
+		(dnp yes)
 		(property "Reference" "C301"
 			(at 145.796 44.45 0)
@@
 		)
 		(property "Part Number" "C0805C104K5RACTU"
+			(at 144.78 46.99 0)
+			(effects
+				(font
+					(size 1.27 1.27)
+				)
+				(hide yes)
+			)
+		)
+		(property "Var" "Assembly Full(+!) Partial(-!)"
 			(at 144.78 46.99 0)
 			(effects
@@
 		)
 		(property "Part Number" "C0603C106M9PAC7411"
+			(at 156.21 46.99 0)
+			(effects
+				(font
+					(size 1.27 1.27)
+				)
+				(hide yes)
+			)
+		)
+		(property "Var" "Assembly Full(-!) Partial(+!)"
 			(at 156.21 46.99 0)
 			(effects
@@
 		(unit 1)
 		(exclude_from_sim no)
-		(in_bom yes)
-		(on_board yes)
-		(dnp no)
+		(in_bom no)
+		(on_board yes)
+		(dnp yes)
 		(fields_autoplaced yes)
 		(property "Reference" "R303"
@@
 		(property "Part Number" "RC0603FR-071KL"
 			(at 205.74 60.96 90)
+			(effects
+				(font
+					(size 1.27 1.27)
+				)
+				(hide yes)
+			)
+		)
+		(property "Var" "Assembly Full(+!) Partial(-!)"
+			(at 205.74 60.96 0)
 			(effects
 				(font
@@
 		(unit 1)
 		(exclude_from_sim no)
-		(in_bom yes)
-		(on_board yes)
-		(dnp no)
+		(in_bom no)
+		(on_board yes)
+		(dnp yes)
 		(fields_autoplaced yes)
 		(property "Reference" "R302"
@@
 			)
 		)
+		(property "Var" "Assembly Full(+!) Partial(-!)"
+			(at 185.42 52.07 0)
+			(effects
+				(font
+					(size 1.27 1.27)
+				)
+				(hide yes)
+			)
+		)
 		(pin "2"
 		)
@@
 		(unit 1)
 		(exclude_from_sim no)
-		(in_bom yes)
-		(on_board yes)
-		(dnp no)
+		(in_bom no)
+		(on_board yes)
+		(dnp yes)
 		(fields_autoplaced yes)
 		(property "Reference" "R301"
@@
 		)
 		(property "Part Number" "RC0603FR-0710KL"
+			(at 137.16 52.07 0)
+			(effects
+				(font
+					(size 1.27 1.27)
+				)
+				(hide yes)
+			)
+		)
+		(property "Var" "Assembly Full(+!) Partial(-!)"
 			(at 137.16 52.07 0)
 			(effects
@@
 		(unit 1)
 		(exclude_from_sim no)
-		(in_bom yes)
-		(on_board yes)
-		(dnp no)
+		(in_bom no)
+		(on_board yes)
+		(dnp yes)
 		(property "Reference" "U301"
 			(at 165.1 54.864 0)
@@
 		)
 		(property "Part Number" "ESP32-WROOM-32E-H4"
+			(at 162.56 91.44 0)
+			(effects
+				(font
+					(size 1.27 1.27)
+				)
+				(hide yes)
+			)
+		)
+		(property "Var" "Assembly Full(+!) Partial(-!)"
 			(at 162.56 91.44 0)
 			(effects
@@
 		(in_bom yes)
 		(on_board yes)
-		(dnp yes)
+		(dnp no)
 		(fields_autoplaced yes)
 		(property "Reference" "J301"
@@
 		)
 		(property "Part Number" "613012243121"
+			(at 107.95 63.5 0)
+			(effects
+				(font
+					(size 1.27 1.27)
+				)
+				(hide yes)
+			)
+		)
+		(property "Var" "Assembly Full(-!) Partial(+!)"
 			(at 107.95 63.5 0)
 			(effects
@@
 		(unit 1)
 		(exclude_from_sim no)
-		(in_bom yes)
-		(on_board yes)
-		(dnp no)
+		(in_bom no)
+		(on_board yes)
+		(dnp yes)
 		(fields_autoplaced yes)
 		(property "Reference" "J303"
@@
 			(at 232.41 63.5 0)
 			(effects
+				(font
+					(size 1.27 1.27)
+				)
+				(hide yes)
+			)
+		)
+		(property "Var" "Assembly Full(+!) Partial(-!)"
+			(at 232.41 63.5 0)
+			(effects

Commit message: cleanup
Parts:
- C301, J303, R301, R302, R303, U301: now fitted; now in the parts list
- C302, J301: now not fitted; now left out of the parts list
Changed lines of the file:
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@@
 		(unit 1)
 		(exclude_from_sim no)
-		(in_bom no)
-		(on_board yes)
-		(dnp yes)
+		(in_bom yes)
+		(on_board yes)
+		(dnp no)
 		(property "Reference" "C301"
 			(at 145.796 44.45 0)
@@
 		(unit 1)
 		(exclude_from_sim no)
-		(in_bom yes)
-		(on_board yes)
-		(dnp no)
+		(in_bom no)
+		(on_board yes)
+		(dnp yes)
 		(property "Reference" "C302"
 			(at 157.48 44.196 0)
@@
 		(unit 1)
 		(exclude_from_sim no)
-		(in_bom no)
-		(on_board yes)
-		(dnp yes)
+		(in_bom yes)
+		(on_board yes)
+		(dnp no)
 		(fields_autoplaced yes)
 		(property "Reference" "R303"
@@
 		(unit 1)
 		(exclude_from_sim no)
-		(in_bom no)
-		(on_board yes)
-		(dnp yes)
+		(in_bom yes)
+		(on_board yes)
+		(dnp no)
 		(fields_autoplaced yes)
 		(property "Reference" "R302"
@@
 		(unit 1)
 		(exclude_from_sim no)
-		(in_bom no)
-		(on_board yes)
-		(dnp yes)
+		(in_bom yes)
+		(on_board yes)
+		(dnp no)
 		(fields_autoplaced yes)
 		(property "Reference" "R301"
@@
 		(unit 1)
 		(exclude_from_sim no)
-		(in_bom no)
-		(on_board yes)
-		(dnp yes)
+		(in_bom yes)
+		(on_board yes)
+		(dnp no)
 		(property "Reference" "U301"
 			(at 165.1 54.864 0)
@@
 		(unit 1)
 		(exclude_from_sim no)
-		(in_bom yes)
-		(on_board yes)
-		(dnp no)
+		(in_bom no)
+		(on_board yes)
+		(dnp yes)
 		(fields_autoplaced yes)
 		(property "Reference" "J301"
@@
 		(unit 1)
 		(exclude_from_sim no)
-		(in_bom no)
-		(on_board yes)
-		(dnp yes)
+		(in_bom yes)
+		(on_board yes)
+		(dnp no)
 		(fields_autoplaced yes)
 		(property "Reference" "J303"
